Commit message: rename mycobot_urdf to have a xacro extension

File: urdf/mycobot_urdf.xacro (robot description, xacro)
@@ -1,3 +1,3 @@
-<?xml version="1.0"?>
+<?xml version="1.0" encoding="utf-8"?>
 <robot  xmlns:xacro="http://www.ros.org/wiki/xacro" name="firefighter" >
 <xacro:property name="width" value=".2" />
@@ -36,5 +36,5 @@
     </visual>
   </link>
-<link name="joint5">
+  <link name="joint5">
     <visual>
       <geometry>
@@ -63,5 +63,5 @@
     </visual>
   </link>
-    <joint name="joint2_to_joint1" type="revolute">
+  <joint name="joint2_to_joint1" type="revolute">
     <axis xyz="0 0 1"/>
     <limit effort = "1000.0" lower = "-3.14" upper = "3.14159" velocity = "0"/>
