Commit message: Update mycobot_urdf.urdf

File: urdf/mycobot_urdf.urdf (robot description, URDF)
Before this commit: robot firefighter, 7 links, 6 joints
Links:
- link joint1: geometry visual mesh filename=package://myCobotROS/urdf/joint1.dae
- link joint2: geometry visual mesh filename=package://myCobotROS/urdf/joint2.dae
- link joint3: geometry visual mesh filename=package://myCobotROS/urdf/joint3.dae
- link joint4: geometry visual mesh filename=package://myCobotROS/urdf/joint4.dae
- link joint5: geometry visual mesh filename=package://myCobotROS/urdf/joint5.dae
- link joint6: geometry visual mesh filename=package://myCobotROS/urdf/joint6.dae

Commit message: Created a realistic texture, changed to dae.

File: urdf/mycobot_urdf.urdf (robot description, URDF)
Before this commit: robot firefighter, 7 links, 6 joints
Links:
- link joint6_flange: geometry visual mesh filename=package://myCobotROS/urdf/joint7.dae
Joints:
- joint joint6_to_joint5: origin xyz=0.0288 0 0.02976 rpy=0 0 0 -> xyz=0.0298 0 0.02876 rpy=0 0 0
- joint joint6output_to_joint6: origin xyz=0 0.0456 0.03792  rpy=0 0 0 -> xyz=0 0.0351 0.03792 rpy=-1.570795 0 0

Commit message: fix: #13 end rotation axis error

File: urdf/mycobot_urdf.urdf (robot description, URDF)
Before this commit: robot firefighter, 7 links, 6 joints
Joints:
- joint joint6output_to_joint6: axis 0 1  0 -> 0 0 1

Commit message: fix: urdf fixed.

File: urdf/mycobot_urdf.urdf (robot description, URDF)
Before this commit: robot firefighter, 7 links, 6 joints
Joints:
- joint joint2_to_joint1: origin xyz=0 0 0.0706 rpy=0 0 0 -> xyz=0 0 0.13156 rpy=0 0 0
- joint joint3_to_joint2: axis 1 0 0 -> 0 0 1; origin xyz=0.03256 0  0.05976 rpy=0 0 0 -> xyz=0 0  0 rpy=0 1.5708 -1.5708
- joint joint4_to_joint3: axis 1 0 0 ->  0 0 1; origin xyz= 0.00272 0 0.1104    rpy=0 0 0 -> xyz=  -0.1104 0 0    rpy=0 0 0
- joint joint5_to_joint4: axis 1 0 0 ->  0 0 1; origin xyz=-0.00164 0 0.096 rpy=0 0 0 -> xyz=-0.096 0 0.06462 rpy=0 0 -1.5708
- joint joint6_to_joint5: origin xyz=0.0298 0 0.02876 rpy=0 0 0 -> xyz=0 -0.07318 0 rpy=1.5708 -1.5708 0
- joint joint6output_to_joint6: origin xyz=0 0.0351 0.03792 rpy=-1.570795 0 0 -> xyz=0 0.0456 0 rpy=-1.5708 0 0

Commit message: fix some scripts for ros noetic

File: urdf/mycobot_urdf.urdf (robot description, URDF)
Before this commit: robot firefighter, 7 links, 6 joints
Links:
- link joint1: geometry visual mesh filename=package://mycobot_ros/urdf/joint1.dae
- link joint2: geometry visual mesh filename=package://mycobot_ros/urdf/joint2.dae
- link joint3: geometry visual mesh filename=package://mycobot_ros/urdf/joint3.dae
- link joint4: geometry visual mesh filename=package://mycobot_ros/urdf/joint4.dae
- link joint5: geometry visual mesh filename=package://mycobot_ros/urdf/joint5.dae
- link joint6: geometry visual mesh filename=package://mycobot_ros/urdf/joint6.dae
- link joint6_flange: geometry visual mesh filename=package://mycobot_ros/urdf/joint7.dae

Commit message: add mycobot urdf collision.

File: urdf/mycobot_urdf.urdf (robot description, URDF)
Before this commit: robot firefighter, 7 links, 6 joints
Links:
- link joint1: geometry collision cylinder length=0.065 radius=0.045; visual mesh filename=package://mycobot_ros/urdf/joint1.dae
- link joint2: geometry collision cylinder length=0.075 radius=0.024; visual mesh filename=package://mycobot_ros/urdf/joint2.dae
- link joint3: geometry collision cylinder length=0.146 radius=0.024; visual mesh filename=package://mycobot_ros/urdf/joint3.dae
- link joint4: geometry collision cylinder length=0.128 radius=0.024; visual mesh filename=package://mycobot_ros/urdf/joint4.dae
- link joint5: geometry collision cylinder length=0.05 radius=0.024; visual mesh filename=package://mycobot_ros/urdf/joint5.dae
- link joint6: geometry collision cylinder length=0.058 radius=0.02; visual mesh filename=package://mycobot_ros/urdf/joint6.dae
- link joint6_flange: geometry collision cylinder length=0.01 radius=0.02; visual mesh filename=package://mycobot_ros/urdf/joint7.dae

Commit message: added mycobot-600 urdf.

File: urdf/mycobot_urdf.urdf (robot description, URDF)
Before this commit: robot firefighter, 7 links, 6 joints
Links:
- link joint1: geometry collision mesh filename=package://mycobot_ros/urdf/joint1.dae; visual mesh filename=package://mycobot_ros/urdf/joint1.dae
- link joint2: geometry collision mesh filename=package://mycobot_ros/urdf/joint2.dae; visual mesh filename=package://mycobot_ros/urdf/joint2.dae
- link joint3: geometry collision mesh filename=package://mycobot_ros/urdf/joint3.dae; visual mesh filename=package://mycobot_ros/urdf/joint3.dae
- link joint4: geometry collision mesh filename=package://mycobot_ros/urdf/joint4.dae; visual mesh filename=package://mycobot_ros/urdf/joint4.dae
- link joint5: geometry collision mesh filename=package://mycobot_ros/urdf/joint5.dae; visual mesh filename=package://mycobot_ros/urdf/joint5.dae
- link joint6: geometry collision mesh filename=package://mycobot_ros/urdf/joint6.dae; visual mesh filename=package://mycobot_ros/urdf/joint6.dae
- link joint6_flange: geometry collision mesh filename=package://mycobot_ros/urdf/joint7.dae; visual mesh filename=package://mycobot_ros/urdf/joint7.dae
