Commit message: add slider control script for pro 600.

File: urdf/600_urdf/mycobot_600_urdf.urdf (robot description, URDF)
Before this commit: robot firefighter, 7 links, 6 joints
Joints:
- joint joint3_to_joint2: axis 0 0 1 -> 0 0 -1; origin xyz=0 0  0 rpy=0 -1.57080  1.57080 -> xyz=0 0  0 rpy=1.5708 0 0
- joint joint4_to_joint3: axis  0 0 1 ->  0 0 -1
- joint joint5_to_joint4: axis  0 0 1 ->  0 0 -1; origin xyz=0.25 0  0.1091 rpy=0 0 1.57080 -> xyz=0.25 0  0.1091 rpy=0 0 0

Commit message: fix 600 model initialize position.

File: urdf/600_urdf/mycobot_600_urdf.urdf (robot description, URDF)
Before this commit: robot firefighter, 7 links, 6 joints
Joints:
- joint joint5_to_joint4: origin xyz=0.25 0  0.1091 rpy=0 0 0 -> xyz=0.25 0  -0.1091 rpy=0 0 0
- joint joint6output_to_joint6: axis 1 0 0 -> -1 0 0; origin xyz=0.07586 0 0 rpy=-1.57080 0 0  -> xyz=-0.07586 0 0 rpy=-1.57080 0 0 
