Commit message: chore: modify dict structure.

File: urdf/mycobot/mycobot_urdf.urdf (robot description, URDF)
Before this commit: robot firefighter, 7 links, 6 joints
Links:
- link joint1: geometry collision mesh filename=package://mycobot_ros/urdf/mycobot/joint1.dae; visual mesh filename=package://mycobot_ros/urdf/mycobot/joint1.dae
- link joint2: geometry collision mesh filename=package://mycobot_ros/urdf/mycobot/joint2.dae; visual mesh filename=package://mycobot_ros/urdf/mycobot/joint2.dae
- link joint3: geometry collision mesh filename=package://mycobot_ros/urdf/mycobot/joint3.dae; visual mesh filename=package://mycobot_ros/urdf/mycobot/joint3.dae
- link joint4: geometry collision mesh filename=package://mycobot_ros/urdf/mycobot/joint4.dae; visual mesh filename=package://mycobot_ros/urdf/mycobot/joint4.dae
- link joint5: geometry collision mesh filename=package://mycobot_ros/urdf/mycobot/joint5.dae; visual mesh filename=package://mycobot_ros/urdf/mycobot/joint5.dae
- link joint6: geometry collision mesh filename=package://mycobot_ros/urdf/mycobot/joint6.dae; visual mesh filename=package://mycobot_ros/urdf/mycobot/joint6.dae
- link joint6_flange: geometry collision mesh filename=package://mycobot_ros/urdf/mycobot/joint7.dae; visual mesh filename=package://mycobot_ros/urdf/mycobot/joint7.dae
