Commit message: feat: add moveit files of mycobot pro 320

File: urdf/320_urdf/mycobot_pro_320.urdf (robot description, URDF)
Before this commit: robot firefighter, 7 links, 6 joints
Links:
- link base: geometry collision cylinder length=0.102 radius=0.0725; visual mesh filename=package://mycobot_ros/urdf/320_urdf/base.dae
- link link1: geometry collision cylinder length=0.106 radius=0.043; visual mesh filename=package://mycobot_ros/urdf/320_urdf/link1.dae
- link link2: geometry collision cylinder length=0.21 radius=0.036; visual mesh filename=package://mycobot_ros/urdf/320_urdf/link2.dae
- link link3: geometry collision cylinder length=0.119 radius=0.0305; visual mesh filename=package://mycobot_ros/urdf/320_urdf/link3.dae
- link link4: geometry collision cylinder length=0.085 radius=0.029; visual mesh filename=package://mycobot_ros/urdf/320_urdf/link4.dae
- link link5: geometry collision cylinder length=0.0849 radius=0.029; visual mesh filename=package://mycobot_ros/urdf/320_urdf/link5.dae
- link link6: geometry collision cylinder length=0.0225 radius=0.026; visual cylinder length=0.02 radius=0.026

Commit message: update pro urdf collision.

File: urdf/320_urdf/mycobot_pro_320.urdf (robot description, URDF)
Before this commit: robot firefighter, 7 links, 6 joints
Links:
- link link2: geometry collision cylinder length=0.18 radius=0.036; visual mesh filename=package://mycobot_ros/urdf/320_urdf/link2.dae
- link link3: geometry collision cylinder length=0.14 radius=0.0305; visual mesh filename=package://mycobot_ros/urdf/320_urdf/link3.dae
- link link4: geometry collision cylinder length=0.083 radius=0.029; visual mesh filename=package://mycobot_ros/urdf/320_urdf/link4.dae

Commit message: feat: added gripper model of pro 320.

File: urdf/320_urdf/mycobot_pro_320.urdf (robot description, URDF)
Before this commit: robot firefighter, 7 links, 6 joints
Links:
- added link gripper; visual mesh filename=package://mycobot_ros/urdf/320_urdf/gripper_ag.dae
Joints:
- added joint gitpper_to_joint6output: type fixed, parent link6, child gripper, origin xyz=0 0 0 rpy=0 0 0 , axis 0 0 1, limit lower=-3.14 upper=3.14159 effort=1000.0 velocity=0

Commit message: fix launch file error.

File: urdf/320_urdf/mycobot_pro_320.urdf (robot description, URDF)
Before this commit: robot firefighter, 8 links, 7 joints
Links:
- link gripper: geometry visual mesh filename=package://mycobot_ros/urdf/320_urdf/gripper.dae

Commit message: update version.

File: urdf/320_urdf/mycobot_pro_320.urdf (robot description, URDF)
Before this commit: robot firefighter, 8 links, 7 joints
Joints:
- joint gitpper_to_joint6output: axis 0 0 1 -> 0 0 0
