Commit message: fix urdf.

File: mycobot_description/urdf/mycobot/mycobot_with_vision copy.urdf (robot description, URDF)
Before this commit: robot mycobot_ai, 1 links, 1 joints
Links:
- link env: geometry visual mesh filename=package://mycobot_description/urdf/mycobot/210110_6000_001_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

File: mycobot_description/urdf/mycobot/mycobot_with_vision.urdf (robot description, URDF)
Before this commit: robot mycobot_ai, 8 links, 7 joints
Links:
- link env: geometry visual mesh filename=package://mycobot_description/urdf/mycobot/210110_6000_001_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
- link joint1: geometry collision mesh filename=package://mycobot_description/urdf/mycobot/joint1.dae; visual mesh filename=package://mycobot_description/urdf/mycobot/joint1.dae
- link joint2: geometry collision mesh filename=package://mycobot_description/urdf/mycobot/joint2.dae; visual mesh filename=package://mycobot_description/urdf/mycobot/joint2.dae
- link joint3: geometry collision mesh filename=package://mycobot_description/urdf/mycobot/joint3.dae; visual mesh filename=package://mycobot_description/urdf/mycobot/joint3.dae
- link joint4: geometry collision mesh filename=package://mycobot_description/urdf/mycobot/joint4.dae; visual mesh filename=package://mycobot_description/urdf/mycobot/joint4.dae
- link joint5: geometry collision mesh filename=package://mycobot_description/urdf/mycobot/joint5.dae; visual mesh filename=package://mycobot_description/urdf/mycobot/joint5.dae
- link joint6: geometry collision mesh filename=package://mycobot_description/urdf/mycobot/joint6.dae; visual mesh filename=package://mycobot_description/urdf/mycobot/joint6.dae
- link joint6_flange: geometry collision mesh filename=package://mycobot_description/urdf/mycobot/joint7.dae; visual mesh filename=package://mycobot_description/urdf/mycobot/joint7.dae
