Commit message: fix: suit dae model.

File: mycobot_description/urdf/mycobot/mycobot_with_vision.urdf (robot description, URDF)
Before this commit: robot mycobot_ai, 8 links, 7 joints
Links:
- link env: geometry visual mesh filename=package://mycobot_description/urdf/mycobot/suit_env.dae

Commit message: optimize

File: mycobot_description/urdf/mycobot/mycobot_with_vision.urdf (robot description, URDF)
Before this commit: robot mycobot_ai, 8 links, 7 joints
Links:
- link env: geometry visual mesh filename=package://mycobot_description/urdf/mycobot/suit_env.dae scale=1.2 1.2 1.2
