Commit message: update

File: mycobot_description/urdf/mycobot/mycobot_with_gripper_parallel.urdf (robot description, URDF)
Before this commit: robot firefighter, 14 links, 13 joints
Joints:
- joint gripper_base_to_gripper_right2: mimic joint=gripper_base_to_gripper_right3 multiplier=1.0 offset=0 -> joint=gripper_controller multiplier=1.0 offset=0
- joint gripper_right3_to_gripper_right1: mimic joint=gripper_base_to_gripper_right3 multiplier=-1.0 offset=0 -> joint=gripper_controller multiplier=-1.0 offset=0

File: mycobot_description/urdf/mycobot/mycobot_with_gripper_up.urdf (robot description, URDF)
Before this commit: robot firefighter, 14 links, 13 joints
Joints:
- joint gripper_base_to_gripper_right2: mimic joint=gripper_base_to_gripper_right3 multiplier=1.0 offset=0 -> joint=gripper_controller multiplier=-1.0 offset=0
- joint gripper_right3_to_gripper_right1: mimic joint=gripper_base_to_gripper_right3 multiplier=-1.0 offset=0 -> joint=gripper_controller multiplier=1.0 offset=0

Commit message: update

File: mycobot_description/urdf/mycobot/mycobot_with_gripper_parallel.urdf (robot description, URDF)
Before this commit: robot firefighter, 14 links, 13 joints
Joints:
- joint gripper_base_to_gripper_right2: mimic joint=gripper_controller multiplier=1.0 offset=0 -> joint=gripper_controller multiplier=-1.0 offset=0
- joint gripper_right3_to_gripper_right1: mimic joint=gripper_controller multiplier=-1.0 offset=0 -> joint=gripper_controller multiplier=1.0 offset=0

Commit message: add 280 G_base.dae

File: mycobot_description/urdf/mycobot/mycobot_with_gripper_parallel.urdf (robot description, URDF)
Before this commit: robot firefighter, 14 links, 13 joints
Links:
- added link g_base; collision mesh filename=package://mycobot_description/urdf/mycobot/G_base.dae; visual mesh filename=package://mycobot_description/urdf/mycobot/G_base.dae
Joints:
- added joint g_base_to_joint1: type fixed, parent g_base, child joint1, origin xyz=0 0 0 rpy=0 0 0, axis 0 0 0, limit lower=-3.14 upper=3.14159 effort=1000.0 velocity=0

File: mycobot_description/urdf/mycobot/mycobot_with_gripper_up.urdf (robot description, URDF)
Before this commit: robot firefighter, 14 links, 13 joints
Links:
- added link g_base; collision mesh filename=package://mycobot_description/urdf/mycobot/G_base.dae; visual mesh filename=package://mycobot_description/urdf/mycobot/G_base.dae
Joints:
- added joint g_base_to_joint1: type fixed, parent g_base, child joint1, origin xyz=0 0 0 rpy=0 0 0, axis 0 0 0, limit lower=-3.14 upper=3.14159 effort=1000.0 velocity=0

Commit message: update urdf

File: mycobot_description/urdf/mycobot/mycobot_with_gripper_parallel.urdf (robot description, URDF)
Before this commit: robot firefighter, 15 links, 14 joints
Joints:
- joint joint2_to_joint1: limit lower=-3.14 upper=3.14159 effort=1000.0 velocity=0 -> lower=-2.879793 upper=2.879793 effort=1000.0 velocity=0
- joint joint3_to_joint2: limit lower=-3.14 upper=3.14159 effort=1000.0 velocity=0 -> lower=-2.879793 upper=2.879793 effort=1000.0 velocity=0
- joint joint4_to_joint3: limit lower=-3.14 upper=3.14159 effort=1000.0 velocity=0 -> lower=-2.879793 upper=2.879793 effort=1000.0 velocity=0
- joint joint5_to_joint4: limit lower=-3.14 upper=3.14159 effort=1000.0 velocity=0 -> lower=-2.879793 upper=2.879793 effort=1000.0 velocity=0
- joint joint6_to_joint5: limit lower=-3.14 upper=3.14159 effort=1000.0 velocity=0 -> lower=-2.879793 upper=2.879793 effort=1000.0 velocity=0
- joint joint6output_to_joint6: limit lower=-3.14 upper=3.14159 effort=1000.0 velocity=0 -> lower=-3.05 upper=3.05 effort=1000.0 velocity=0

File: mycobot_description/urdf/mycobot/mycobot_with_gripper_up.urdf (robot description, URDF)
Before this commit: robot firefighter, 15 links, 14 joints
Joints:
- joint joint2_to_joint1: limit lower=-3.14 upper=3.14159 effort=1000.0 velocity=0 -> lower=-2.879793 upper=2.879793 effort=1000.0 velocity=0
- joint joint3_to_joint2: limit lower=-3.14 upper=3.14159 effort=1000.0 velocity=0 -> lower=-2.879793 upper=2.879793 effort=1000.0 velocity=0
- joint joint4_to_joint3: limit lower=-3.14 upper=3.14159 effort=1000.0 velocity=0 -> lower=-2.879793 upper=2.879793 effort=1000.0 velocity=0
- joint joint5_to_joint4: limit lower=-3.14 upper=3.14159 effort=1000.0 velocity=0 -> lower=-2.879793 upper=2.879793 effort=1000.0 velocity=0
- joint joint6_to_joint5: limit lower=-3.14 upper=3.14159 effort=1000.0 velocity=0 -> lower=-2.879793 upper=2.879793 effort=1000.0 velocity=0
- joint joint6output_to_joint6: limit lower=-3.14 upper=3.14159 effort=1000.0 velocity=0 -> lower=-3.05 upper=3.05 effort=1000.0 velocity=0
