Commit message: Fix urdf joint axis angles to match real robot

File: mycobot_description/urdf/mycobot/mycobot_urdf.urdf (robot description, URDF)
Before this commit: robot firefighter, 7 links, 6 joints
Joints:
- joint joint2_to_joint1: axis 0 0 1 -> 0 0 -1
- joint joint3_to_joint2: axis 0 0 1 -> 0 0 -1
- joint joint5_to_joint4: axis  0 0 1 ->  0 0 -1
- joint joint6_to_joint5: axis 0 0 1 -> 0 0 -1
- joint joint6output_to_joint6: axis 0 0 1 -> 0 0 -1

File: mycobot_description/urdf/mycobot/mycobot_with_vision.urdf (robot description, URDF)
Before this commit: robot mycobot_ai, 8 links, 7 joints
Joints:
- joint joint2_to_joint1: axis 0 0 1 -> 0 0 -1
- joint joint3_to_joint2: axis 0 0 1 -> 0 0 -1
- joint joint5_to_joint4: axis  0 0 1 ->  0 0 -1
- joint joint6_to_joint5: axis 0 0 1 -> 0 0 -1
- joint joint6output_to_joint6: axis 0 0 1 -> 0 0 -1

Commit message: Update mycobot_urdf.urdf

File: mycobot_description/urdf/mycobot/mycobot_urdf.urdf (robot description, URDF)
Before this commit: robot firefighter, 8 links, 7 joints
Joints:
- joint g_base_to_joint1: limit lower=-3.14 upper=3.14159 effort=1000.0 velocity=0 -> lower=0 upper=0 effort=1000.0 velocity=1
- joint joint2_to_joint1: limit lower=-3.14 upper=3.14159 effort=1000.0 velocity=0 -> lower=-2.93 upper=2.9321 effort=1000.0 velocity=1
- joint joint3_to_joint2: limit lower=-3.14 upper=3.14159 effort=1000.0 velocity=0 -> lower=-2.36 upper=2.3561 effort=1000.0 velocity=1
- joint joint4_to_joint3: limit lower=-3.14 upper=3.14159 effort=1000.0 velocity=0 -> lower=-2.62 upper=2.6179 effort=1000.0 velocity=0
- joint joint5_to_joint4: limit lower=-3.14 upper=3.14159 effort=1000.0 velocity=0 -> lower=-2.53 upper=2.5307 effort=1000.0 velocity=0
- joint joint6_to_joint5: limit lower=-3.14 upper=3.14159 effort=1000.0 velocity=0 -> lower=-2.88 upper=2.8797 effort=1000.0 velocity=1
- joint joint6output_to_joint6: limit lower=-3.14 upper=3.14159 effort=1000.0 velocity=0 -> lower=-3.14 upper=3.14159 effort=1000.0 velocity=1
