Commit message: fix dae,urdf

File: mycobot_description/urdf/260_urdf/mypal_260.urdf (robot description, URDF)
Before this commit: robot firefighter, 6 links, 5 joints
Links:
- link base: geometry collision mesh filename=package://mycobot_description/urdf/260_urdf/base.dae; visual mesh filename=package://mycobot_description/urdf/260_urdf/base.dae
- link link1: geometry collision mesh filename=package://mycobot_description/urdf/260_urdf/link1.dae; visual mesh filename=package://mycobot_description/urdf/260_urdf/link1.dae
- link link2: geometry collision mesh filename=package://mycobot_description/urdf/260_urdf/link2.dae; visual mesh filename=package://mycobot_description/urdf/260_urdf/link2.dae
- link link3: geometry collision mesh filename=package://mycobot_description/urdf/260_urdf/link3.dae; visual mesh filename=package://mycobot_description/urdf/260_urdf/link3.dae
- link link4: geometry collision mesh filename=package://mycobot_description/urdf/260_urdf/link4.dae; visual mesh filename=package://mycobot_description/urdf/260_urdf/link4.dae
- link link5: geometry collision cylinder length=0.015 radius=0.0152; visual cylinder length=0.015 radius=0.0152
