Commit message: optimize

File: mycobot_description/urdf/260_urdf/mypal_260_aikit.urdf (robot description, URDF)
Before this commit: robot firefighter, 7 links, 6 joints
Joints:
- joint joint3_to_joint2: limit lower=-0.213 upper=1.106 effort=1000.0 velocity=0 -> lower=-0.213 upper=0.872665 effort=1000.0 velocity=0
- joint joint4_to_joint3: axis  0 0 1 -> (none); limit lower=0 upper=1.5707963 effort=1000.0 velocity=0 -> (none)
