Commit message: Remove the gripper of the 320 model

File: mycobot_description/urdf/320_urdf/mycobot_pro_320.urdf (robot description, URDF)
Before this commit: robot firefighter, 8 links, 7 joints
Links:
- removed link gripper
Joints:
- removed joint gitpper_to_joint6output

Commit message: Fix the problem that moveit cannot be used in ubuntu20.04

File: mycobot_description/urdf/320_urdf/mycobot_pro_320.urdf (robot description, URDF)
Before this commit: robot firefighter, 7 links, 6 joints
Links:
- added link gripper; visual mesh filename=package://mycobot_description/urdf/320_urdf/gripper.dae
Joints:
- added joint gitpper_to_joint6output: type fixed, parent link6, child gripper, origin xyz=0 0 0 rpy=0 0 0 , axis 0 0 0, limit lower=-3.14 upper=3.14159 effort=1000.0 velocity=0

Commit message: support mycobot320

File: mycobot_description/urdf/320_urdf/mycobot_pro_320.urdf (robot description, URDF)
Before this commit: robot firefighter, 8 links, 7 joints
Links:
- removed link gripper
- link base: geometry visual mesh filename=package://mycobot_description/urdf/320_urdf/base.dae
- link link1: geometry visual mesh filename=package://mycobot_description/urdf/320_urdf/link1.dae
- link link2: geometry visual mesh filename=package://mycobot_description/urdf/320_urdf/link2.dae
- link link3: geometry visual mesh filename=package://mycobot_description/urdf/320_urdf/link3.dae
- link link4: geometry visual mesh filename=package://mycobot_description/urdf/320_urdf/link4.dae
- link link5: geometry visual mesh filename=package://mycobot_description/urdf/320_urdf/link5.dae
- link link6: geometry visual cylinder length=0.02 radius=0.026
Joints:
- removed joint gitpper_to_joint6output

Commit message: change mycobot_pro_320.urdf

File: mycobot_description/urdf/320_urdf/mycobot_pro_320.urdf (robot description, URDF)
Before this commit: robot firefighter, 8 links, 7 joints
Links:
- removed link gripper
- link base: geometry visual mesh filename=package://mycobot_description/urdf/320_urdf/base.dae
- link link1: geometry visual mesh filename=package://mycobot_description/urdf/320_urdf/link1.dae
- link link2: geometry visual mesh filename=package://mycobot_description/urdf/320_urdf/link2.dae
- link link3: geometry visual mesh filename=package://mycobot_description/urdf/320_urdf/link3.dae
- link link4: geometry visual mesh filename=package://mycobot_description/urdf/320_urdf/link4.dae
- link link5: geometry visual mesh filename=package://mycobot_description/urdf/320_urdf/link5.dae
- link link6: geometry visual mesh filename=package://mycobot_description/urdf/320_urdf/link6.dae
Joints:
- removed joint gitpper_to_joint6output
- joint joint6output_to_joint6: axis 0 0 1 -> 1 0 0; origin xyz=0 0.06 0 rpy=-1.57080 0 0  -> xyz=0.02155 -0.01 -0.034 rpy=1.57080 0 1.57080 

Commit message: fix urdf

File: mycobot_description/urdf/320_urdf/mycobot_pro_320.urdf (robot description, URDF)
Before this commit: robot firefighter, 7 links, 6 joints
Links:
- link base: geometry collision mesh filename=package://mycobot_description/urdf/320_urdf/base.dae; visual mesh filename=package://mycobot_description/urdf/320_urdf/base.dae
- link link1: geometry collision mesh filename=package://mycobot_description/urdf/320_urdf/link1.dae; visual mesh filename=package://mycobot_description/urdf/320_urdf/link1.dae
- link link2: geometry collision mesh filename=package://mycobot_description/urdf/320_urdf/link2.dae; visual mesh filename=package://mycobot_description/urdf/320_urdf/link2.dae
- link link3: geometry collision mesh filename=package://mycobot_description/urdf/320_urdf/link3.dae; visual mesh filename=package://mycobot_description/urdf/320_urdf/link3.dae
- link link4: geometry collision mesh filename=package://mycobot_description/urdf/320_urdf/link4.dae; visual mesh filename=package://mycobot_description/urdf/320_urdf/link4.dae
- link link5: geometry collision mesh filename=package://mycobot_description/urdf/320_urdf/link5.dae; visual mesh filename=package://mycobot_description/urdf/320_urdf/link5.dae
- link link6: geometry collision mesh filename=package://mycobot_description/urdf/320_urdf/link6.dae; visual mesh filename=package://mycobot_description/urdf/320_urdf/link6.dae
Joints:
- joint joint3_to_joint2: origin xyz=0 0  0 rpy=0 -1.57080  1.57080 -> xyz=0 0 0 rpy=0 -1.5708 1.5708
- joint joint5_to_joint4: origin xyz=0.1 0  0.090 rpy=0 0 1.57080 -> xyz=0.1 0 0.09  rpy= 0 0 1.57080
- joint joint6_to_joint5: origin xyz=0 -0.08515 0 rpy=1.57080 -1.57080 0 -> xyz=0 -0.07318 0 rpy=1.5708 -1.5708 0
- joint joint6output_to_joint6: axis 1 0 0 -> 0 0 1; origin xyz=0.02155 -0.01 -0.034 rpy=1.57080 0 1.57080  -> xyz=0.00 0.06635 0 rpy=-1.5708 0 0
