Commit message: add old 320 M5 gripper moveit

File: mycobot_description/urdf/320_urdf/mycobot_pro_320_gripper.urdf (robot description, URDF)
Before this commit: robot firefighter, 14 links, 13 joints
Links:
- added link base_footprint
- link base: mass None -> 0.1
- link gripper_base: mass None -> 0.1
- link gripper_left1: mass None -> 0.1
- link gripper_left2: mass None -> 0.1
- link gripper_left3: mass None -> 0.1
- link gripper_right1: mass None -> 0.1
- link gripper_right2: mass None -> 0.1
- link gripper_right3: mass None -> 0.1
- link link1: mass None -> 0.1
- link link2: mass None -> 0.1
- link link3: mass None -> 0.1
- link link4: mass None -> 0.1
- link link5: mass None -> 0.1
- link link6: mass None -> 0.1
Joints:
- added joint base_footprint_joint: type fixed, parent base_footprint, child base
