Commit message: fix joint2

File: mycobot_description/urdf/mecharm_pi/mecharm_pi.urdf (robot description, URDF)
Before this commit: robot firefighter, 7 links, 6 joints
Joints:
- joint joint3_to_joint2: origin xyz=0.04 -0.096 0    rpy=0 0 0  -> xyz=0.0 -0.1 0    rpy=0 0 0 
- joint joint4_to_joint3: origin xyz=0.1 -0.003  -0.003 rpy=0 1.5708 0  -> xyz=0.108 -0.005  -0.001 rpy=0 1.5708 0 
- joint joint6_to_joint5: origin xyz= 0.06 0.002 -0.0 rpy=  0 1.5708 0  -> xyz= 0.06 0.00 -0.0 rpy=  0 1.5708 0 

Commit message: fix urdf

File: mycobot_description/urdf/mecharm_pi/mecharm_pi.urdf (robot description, URDF)
Before this commit: robot firefighter, 7 links, 6 joints
Joints:
- joint joint2_to_joint1: origin xyz=0 0 0.038 rpy= -1.5708 0 0  -> xyz=0 0 0.038 rpy= 1.5708 0 0 
- joint joint3_to_joint2: origin xyz=0.0 -0.1 0    rpy=0 0 0  -> xyz=0.0 0.1 0    rpy=3.1415926 0 0 
- joint joint5_to_joint4: origin xyz= 0 0 0.0 rpy=  0 -1.5708 0  -> xyz= -0.001 0 0.0 rpy=  0 -1.5708 3.1415926

Commit message: change joint3_joint2 lower

File: mycobot_description/urdf/mecharm_pi/mecharm_pi.urdf (robot description, URDF)
Before this commit: robot firefighter, 7 links, 6 joints
Joints:
- joint joint3_to_joint2: limit lower=-3.14 upper=0.785398 effort=1000.0 velocity=0 -> lower=-3.10 upper=0.785398 effort=1000.0 velocity=0

Commit message: change joint3_joint2 lower

File: mycobot_description/urdf/mecharm_pi/mecharm_pi.urdf (robot description, URDF)
Before this commit: robot firefighter, 7 links, 6 joints
Joints:
- joint joint3_to_joint2: limit lower=-3.10 upper=0.785398 effort=1000.0 velocity=0 -> lower=-3.08 upper=0.785398 effort=1000.0 velocity=0
