Commit message: fix bug

File: mycobot_description/urdf/new_320_urdf/new_mycobot_pro_320moveit.urdf (robot description, URDF)
Before this commit: robot firefighter, 7 links, 6 joints
Joints:
- joint joint3_to_joint2: origin xyz=0 0  0 rpy=0 -1.57080  1.57080 -> xyz=0 0 -0.014 rpy=0 -1.57080  1.57080
- joint joint5_to_joint4: origin xyz=0.12 0  0.090 rpy=0 0 1.57080 -> xyz=0.12 0  0.09 rpy=0 0 1.57080
- joint joint6_to_joint5: origin xyz=0 -0.08515 0 rpy=1.57080 0 0 -> xyz=0 -0.090 0 rpy=1.57080 0 0
- joint joint6output_to_joint6: origin xyz=0 0.0760 0 rpy=-1.57080 0 0  -> xyz=0 0.06635 0 rpy=-1.57080 0 0 
