Commit message: fix urdf

File: mycobot_description/urdf/new_320_urdf/new_mycobot_pro_320.urdf (robot description, URDF)
Before this commit: robot firefighter, 7 links, 6 joints
Joints:
- joint joint2_to_joint1: origin xyz=0 0 0.16846 rpy=0 0 0 -> xyz=0 0 0.17846 rpy=0 0 0
- joint joint3_to_joint2: origin xyz=0 0 0 rpy=0 -1.5708 1.5708 -> xyz=0 0 -0.014 rpy=0 -1.5708 1.5708
- joint joint6_to_joint5: origin xyz=0 -0.080 0 rpy=1.5708 0 0 -> xyz=0 -0.090 0.0 rpy=1.5708 0 0
- joint joint6output_to_joint6: origin xyz=0 0.0760 0 rpy=-1.5708 0 0 -> xyz=0 0.06635 0.0 rpy=-1.5708 0 0

Commit message: update new_320_M5 urdf

File: mycobot_description/urdf/new_320_urdf/new_mycobot_pro_320.urdf (robot description, URDF)
Before this commit: robot firefighter, 7 links, 6 joints
Joints:
- joint joint2_to_joint1: limit lower=-3.14 upper=3.14159 effort=1000.0 velocity=0 -> lower=-2.96 upper=2.96 effort=1000.0 velocity=0; origin xyz=0 0 0.17846 rpy=0 0 0 -> xyz=0 0 0.162 rpy=0 0 0
- joint joint3_to_joint2: limit lower=-3.14 upper=3.14159 effort=1000.0 velocity=0 -> lower=-2.79 upper=2.79 effort=1000.0 velocity=0; origin xyz=0 0 -0.014 rpy=0 -1.5708 1.5708 -> xyz=0 0 0 rpy=0 -1.5708 1.5708
- joint joint4_to_joint3: limit lower=-3.14 upper=3.14159 effort=1000.0 velocity=0 -> lower=-2.79 upper=2.79 effort=1000.0 velocity=0
- joint joint5_to_joint4: limit lower=-3.14 upper=3.14159 effort=1000.0 velocity=0 -> lower=-2.79 upper=2.79 effort=1000.0 velocity=0; origin xyz=0.12 0 0.09  rpy= 0 0 1.57080 -> xyz=0.1205 0 0.082  rpy= 0 0 1.57080
- joint joint6_to_joint5: limit lower=-3.14 upper=3.14159 effort=1000.0 velocity=0 -> lower=-2.96 upper=2.96 effort=1000.0 velocity=0; origin xyz=0 -0.090 0.0 rpy=1.5708 0 0 -> xyz=0 -0.084 0.0 rpy=1.5708 0 0
- joint joint6output_to_joint6: limit lower=-3.14 upper=3.14159 effort=1000.0 velocity=0 -> lower=-3.05 upper=3.05 effort=1000.0 velocity=0

File: mycobot_description/urdf/new_320_urdf/new_mycobot_pro_320moveit.urdf (robot description, URDF)
Before this commit: robot firefighter, 7 links, 6 joints
Joints:
- joint joint2_to_joint1: limit lower=-3.14 upper=3.14159 effort=1000.0 velocity=0 -> lower=-2.96 upper=2.96 effort=1000.0 velocity=0; origin xyz=0 0 0.17846 rpy=0 0 0 -> xyz=0 0 0.162 rpy=0 0 0
- joint joint3_to_joint2: limit lower=-3.14 upper=3.14159 effort=1000.0 velocity=0 -> lower=-2.79 upper=2.79 effort=1000.0 velocity=0; origin xyz=0 0 -0.014 rpy=0 -1.57080  1.57080 -> xyz=0 0 0 rpy=0 -1.57080  1.57080
- joint joint4_to_joint3: limit lower=-3.14 upper=3.14159 effort=1000.0 velocity=0 -> lower=-2.79 upper=2.79 effort=1000.0 velocity=0
- joint joint5_to_joint4: limit lower=-3.14 upper=3.14159 effort=1000.0 velocity=0 -> lower=-2.79 upper=2.79 effort=1000.0 velocity=0; origin xyz=0.12 0  0.09 rpy=0 0 1.57080 -> xyz=0.1205 0  0.082 rpy=0 0 1.57080
- joint joint6_to_joint5: limit lower=-3.14 upper=3.14159 effort=1000.0 velocity=0 -> lower=-2.96 upper=2.96 effort=1000.0 velocity=0; origin xyz=0 -0.090 0 rpy=1.57080 0 0 -> xyz=0 -0.084 0 rpy=1.57080 0 0
- joint joint6output_to_joint6: limit lower=-3.14 upper=3.14159 effort=1000.0 velocity=0 -> lower=-3.05 upper=3.05 effort=1000.0 velocity=0
