Commit message: fix mycobot_600_urdf

File: mycobot_description/urdf/600_urdf/mycobot_600_urdf.urdf (robot description, URDF)
Before this commit: robot firefighter, 7 links, 6 joints
Joints:
- joint joint3_to_joint2: axis 0 0 -1 -> 0 0 1; limit lower=-3.14 upper=3.14159 effort=1000.0 velocity=0 -> lower=-4.71 upper=1.5708 effort=1000.0 velocity=0; origin xyz=0 0  0 rpy=1.5708 0 0 -> xyz=0 0  0 rpy=1.5708 -1.5708 0
- joint joint4_to_joint3: axis  0 0 -1 ->  0 0 1; limit lower=-3.14 upper=3.14159 effort=1000.0 velocity=0 -> lower=-2.61 upper=2.618 effort=1000.0 velocity=0
- joint joint5_to_joint4: limit lower=-3.14 upper=3.14159 effort=1000.0 velocity=0 -> lower=-4.53 upper=1.3962 effort=1000.0 velocity=0; origin xyz=0.25 0  -0.1091 rpy=0 0 0 -> xyz=0.25 0  -0.1091 rpy=0 0 1.5708
- joint joint6_to_joint5: limit lower=-3.14 upper=3.14159 effort=1000.0 velocity=0 -> lower=-2.93 upper=2.9321 effort=1000.0 velocity=0
- joint joint6output_to_joint6: limit lower=-3.14 upper=3.14159 effort=1000.0 velocity=0 -> lower=-3.03 upper=3.0368 effort=1000.0 velocity=0

Commit message: change urdf

File: mycobot_description/urdf/600_urdf/mycobot_600_urdf.urdf (robot description, URDF)
Before this commit: robot firefighter, 7 links, 6 joints
Joints:
- joint joint3_to_joint2: axis 0 0 1 -> 0 0 -1; origin xyz=0 0  0 rpy=1.5708 -1.5708 0 -> xyz=0 0  0 rpy=1.5708 0 0
- joint joint4_to_joint3: axis  0 0 1 ->  0 0 -1
- joint joint5_to_joint4: origin xyz=0.25 0  -0.1091 rpy=0 0 1.5708 -> xyz=0.25 0  -0.1091 rpy=0 0 0
