Commit message: fix

File: mycobot_description/urdf/260_pi/mypal_260_pi_aikit.urdf (robot description, URDF)
Before this commit: robot firefighter, 6 links, 5 joints
Links:
- added link env; visual mesh filename=package://mycobot_description/urdf/260_pi/suit_env.dae scale=1.2 1.2 1.2
Joints:
- added joint vision_joint: type fixed, parent base, child env, origin xyz=0 0 0 rpy=0 0 0, axis 0 0 0, limit lower=-3.14 upper=3.14159 effort=1000.0 velocity=0
