Commit message: edit urdf

File: mycobot_description/urdf/mybuddy/mybuddy.urdf (robot description, URDF)
Before this commit: robot firefighter, 9 links, 8 joints
Links:
- added link link2_L; collision mesh filename=package://mycobot_description/urdf/mybuddy/joint2_L.dae; visual mesh filename=package://mycobot_description/urdf/mybuddy/joint2_L.dae
- added link link3_L; collision mesh filename=package://mycobot_description/urdf/mybuddy/joint3_L.dae; visual mesh filename=package://mycobot_description/urdf/mybuddy/joint3_L.dae
- added link link4_L; collision mesh filename=package://mycobot_description/urdf/mybuddy/joint4_L.dae; visual mesh filename=package://mycobot_description/urdf/mybuddy/joint4_L.dae
- added link link5_L; collision mesh filename=package://mycobot_description/urdf/mybuddy/joint5_L.dae; visual mesh filename=package://mycobot_description/urdf/mybuddy/joint5_L.dae
- added link link6_L; collision mesh filename=package://mycobot_description/urdf/mybuddy/joint6_L.dae; visual mesh filename=package://mycobot_description/urdf/mybuddy/joint6_L.dae
Joints:
- added joint joint2_L: type revolute, parent link1_L, child link2_L, origin xyz= 0 -0.05 0.00   rpy=1.5708 -1.5708 0, axis  0 0 1, limit lower=-3.14 upper=3.14159 effort=1000.0 velocity=0
- added joint joint3_L: type revolute, parent link2_L, child link3_L, origin xyz= 0.11 0.0 0.00   rpy=0 0 0, axis  0 0 1, limit lower=-3.14 upper=3.14159 effort=1000.0 velocity=0
- added joint joint4_L: type revolute, parent link3_L, child link4_L, origin xyz= 0.097 0.0 -0.0   rpy=0 0 1.5708, axis  0 0 1, limit lower=-3.14 upper=3.14159 effort=1000.0 velocity=0
- added joint joint5_L: type revolute, parent link4_L, child link5_L, origin xyz=0 -0.035  0.00   rpy=1.5708 3.14159 0 , axis  0 0 1, limit lower=-3.14 upper=3.14159 effort=1000.0 velocity=0
- added joint joint6_L: type revolute, parent link5_L, child link6_L, origin xyz=-0.035 0 0.0375   rpy=0 -1.5708 0, axis  0 0 1, limit lower=-3.14 upper=3.14159 effort=1000.0 velocity=0
- joint joint1_L: origin xyz= 0 0.129 0.001    rpy=1.5708 0 0 -> xyz= 0 -0.129 0.001    rpy=1.5708 -1.5708 0
- joint joint1_R: origin xyz= 0 -0.129 0.001    rpy=1.5708 0 0 -> xyz= 0 0.129 0.001    rpy=-1.5708 3.14159 0
- joint joint2_R: origin xyz= 0 -0.05 0.00   rpy=1.5708 0 0 -> xyz=-0.05 0.00 0.00   rpy=0 -1.5708 0
- joint joint4_R: origin xyz= 0.097 0.0 -0.0   rpy=0 0 0 -> xyz= 0.097 0.0 -0.0   rpy=0 0 1.5708
- joint joint5_R: origin xyz= 0.1 0 0.00   rpy=0 0 0 -> xyz=0 -0.035  0.00   rpy=1.570795 0 0
- joint joint6_R: origin xyz= 0.1 0.0 0.00   rpy=0 0 0 -> xyz=-0.035 0 0.0375   rpy=0 -1.5708 0
