Commit message: update mira urdf

File: mycobot_description/urdf/mira_urdf/mira.urdf (robot description, URDF)
Before this commit: robot firefighter, 4 links, 3 joints
Joints:
- joint joint1_to_base: origin xyz=0 0 0.12 rpy=0 0 0 -> xyz=0 0 0.12 rpy=3.1415926 0 0
- joint joint2_to_joint1: limit lower=0 upper=1.5708 effort=1000.0 velocity=0 -> lower=0 upper=1.14 effort=1000.0 velocity=0; origin xyz=0.03 0 -0.01 rpy= -1.5707963 0 0  -> xyz=0.03 0 0.01 rpy= -1.5707963 3.1415926 3.1415926 
- joint joint3_to_joint2: limit lower=0 upper=1.309 effort=1000.0 velocity=0 -> lower=0 upper=1.0472 effort=1000.0 velocity=0; origin xyz=0.004 -0.126 0    rpy=0 0 0  -> xyz=0.00 -0.12 0    rpy=0 0 0 

Commit message: update

File: mycobot_description/urdf/mira_urdf/mira.urdf (robot description, URDF)
Before this commit: robot firefighter, 4 links, 3 joints
Joints:
- joint joint1_to_base: limit lower=-2.967 upper=2.967 effort=1000.0 velocity=0 -> lower=-2.36 upper=2.967 effort=1000.0 velocity=0
- joint joint2_to_joint1: limit lower=0 upper=1.14 effort=1000.0 velocity=0 -> lower=0 upper=0.90 effort=1000.0 velocity=0

Commit message: update

File: mycobot_description/urdf/mira_urdf/mira.urdf (robot description, URDF)
Before this commit: robot firefighter, 4 links, 3 joints
Joints:
- joint joint2_to_joint1: limit lower=0 upper=0.90 effort=1000.0 velocity=0 -> lower=0 upper=1.14 effort=1000.0 velocity=0
