Commit message: update ultraArm angles range

File: mycobot_description/urdf/ultraArm_urdf/ultraArm.urdf (robot description, URDF)
Before this commit: robot firefighter, 4 links, 3 joints
Joints:
- joint joint2_to_joint1: limit lower=0 upper=1.14 effort=1000.0 velocity=0 -> lower=-0.31 upper=1.57 effort=1000.0 velocity=0
- joint joint3_to_joint2: limit lower=0 upper=1.0472 effort=1000.0 velocity=0 -> lower=-0.087 upper=1.0472 effort=1000.0 velocity=0
