Commit message: opt myarm urdf and and moveit config

File: mycobot_description/urdf/myarm/myarm_urdf.urdf (robot description, URDF)
Before this commit: robot firefighter, 8 links, 7 joints
Joints:
- joint joint2_to_joint1: origin xyz=0 0  0 rpy=-1.5708 0 0 -> xyz=0 0  0 rpy=1.5708 3.14159 0

Commit message: fix urdf model

File: mycobot_description/urdf/myarm/myarm_urdf.urdf (robot description, URDF)
Before this commit: robot firefighter, 8 links, 7 joints
Joints:
- joint joint6_to_joint5: origin xyz=0 0.0 0 rpy=-1.5708 0 0 -> xyz=0 0.0 0 rpy=-1.5708 3.14 0
- joint joint7_to_joint6: origin xyz=0 -0.056 0 rpy=1.5708 0 0 -> xyz=0 0.056 0 rpy=-1.5708 1.5708 0

Commit message: fix and opt urdf

File: mycobot_description/urdf/myarm/myarm_urdf.urdf (robot description, URDF)
Before this commit: robot firefighter, 8 links, 7 joints
Joints:
- joint joint6_to_joint5: origin xyz=0 0.0 0 rpy=-1.5708 3.14 0 -> xyz=0 0.0 0 rpy=-1.5708 0 0
- joint joint7_to_joint6: origin xyz=0 0.056 0 rpy=-1.5708 1.5708 0 -> xyz=0 -0.056 0 rpy=1.5708 0 0

Commit message: update urdf

File: mycobot_description/urdf/myarm/myarm_urdf.urdf (robot description, URDF)
Before this commit: robot firefighter, 8 links, 7 joints
Joints:
- joint joint1_to_base: limit lower=-3.14 upper=3.14159 effort=1000.0 velocity=0 -> lower=-3.14 upper=3.14 effort=1000.0 velocity=0
- joint joint3_to_joint2: limit lower=-3.14 upper=3.14159 effort=1000.0 velocity=0 -> lower=-3.14 upper=3.14 effort=1000.0 velocity=0
- joint joint5_to_joint4: limit lower=-3.14 upper=3.14159 effort=1000.0 velocity=0 -> lower=-3.14 upper=3.14 effort=1000.0 velocity=0
- joint joint7_to_joint6: limit lower=-3.14 upper=3.14159 effort=1000.0 velocity=0 -> lower=-3.14 upper=3.14 effort=1000.0 velocity=0

Commit message: update myarm_urdf joint limit

File: mycobot_description/urdf/myarm/myarm_urdf.urdf (robot description, URDF)
Before this commit: robot firefighter, 8 links, 7 joints
Joints:
- joint joint1_to_base: limit lower=-3.14 upper=3.14 effort=1000.0 velocity=0 -> lower=-2.79 upper=2.87 effort=1000.0 velocity=0
- joint joint2_to_joint1: limit lower=-1.5708 upper=1.5708 effort=1000.0 velocity=0 -> lower=-1.5708 upper=1.39 effort=1000.0 velocity=0
- joint joint3_to_joint2: limit lower=-3.14 upper=3.14 effort=1000.0 velocity=0 -> lower=-3.05 upper=3.05 effort=1000.0 velocity=0
- joint joint4_to_joint3: limit lower=-1.5708 upper=1.5708 effort=1000.0 velocity=0 -> lower=-1.91 upper=1.39 effort=1000.0 velocity=0
- joint joint5_to_joint4: limit lower=-3.14 upper=3.14 effort=1000.0 velocity=0 -> lower=-2.96 upper=2.96 effort=1000.0 velocity=0
- joint joint6_to_joint5: limit lower=-1.5708 upper=1.5708 effort=1000.0 velocity=0 -> lower=-1.91 upper=1.91 effort=1000.0 velocity=0

Commit message: Change joint limit and J2 movement direction_v20230718

File: mycobot_description/urdf/myarm/myarm_urdf.urdf (robot description, URDF)
Before this commit: robot firefighter, 8 links, 7 joints
Joints:
- joint joint1_to_base: limit lower=-2.79 upper=2.87 effort=1000.0 velocity=0 -> lower=-2.7925 upper=2.7925 effort=1000.0 velocity=0
- joint joint2_to_joint1: limit lower=-1.5708 upper=1.39 effort=1000.0 velocity=0 -> lower=-1.3962 upper=1.3962 effort=1000.0 velocity=0; origin xyz=0 0  0 rpy=1.5708 3.14159 0 -> xyz=0 0  0 rpy=-1.5708 0 0
- joint joint3_to_joint2: limit lower=-3.05 upper=3.05 effort=1000.0 velocity=0 -> lower=-2.8797 upper=2.8797 effort=1000.0 velocity=0
- joint joint4_to_joint3: limit lower=-1.91 upper=1.39 effort=1000.0 velocity=0 -> lower=-1.7453 upper=1.3962 effort=1000.0 velocity=0; origin xyz=0.0 0 0.0 rpy=-1.5708 0 0 -> xyz=0.0 0 0.0 rpy=-1.5708 0 3.14159
- joint joint5_to_joint4: limit lower=-2.96 upper=2.96 effort=1000.0 velocity=0 -> lower=-2.8797 upper=2.8797 effort=1000.0 velocity=0
- joint joint6_to_joint5: limit lower=-1.91 upper=1.91 effort=1000.0 velocity=0 -> lower=-1.9198 upper=1.9198 effort=1000.0 velocity=0
- joint joint7_to_joint6: limit lower=-3.14 upper=3.14 effort=1000.0 velocity=0 -> lower=-2.8797 upper=2.8797 effort=1000.0 velocity=0
