Commit message: add aikit-320 ros

File: mycobot_description/urdf/new_320_pi/new_mycobot_vision_v2.urdf (robot description, URDF)
Before this commit: robot firefighter, 7 links, 6 joints
Links:
- added link env; visual mesh filename=package://mycobot_description/urdf/new_320_pi/ai_kit320.dae
Joints:
- added joint vision_joint: type fixed, parent base, child env, origin xyz=0 0 0 rpy=0 0 0, axis 0 0 0, limit lower=-3.14 upper=3.14159 effort=1000.0 velocity=0

Commit message: update 2022 version 320 ROS1 urdf model file

File: mycobot_description/urdf/new_320_pi/new_mycobot_vision_v2.urdf (robot description, URDF)
Before this commit: robot firefighter, 8 links, 7 joints
Joints:
- joint joint2_to_joint1: origin xyz=0 0 0.162 rpy=0 0 0 -> xyz=0 0 0.173 rpy=0 0 0
- joint joint3_to_joint2: origin xyz=0 0 0 rpy=0 -1.5708 1.5708 -> xyz=0 -0.086 0 rpy=0 -1.5708 1.5708
- joint joint4_to_joint3: origin xyz=0.13635 0 0    rpy=0 0 0 -> xyz=0.13635 0 -0.086    rpy=0 0 0
- joint joint5_to_joint4: origin xyz=0.1205 0 0.082  rpy= 0 0 1.57080 -> xyz=0.1195 0 0.082  rpy= 0 0 1.57080
- joint joint6_to_joint5: origin xyz=0 -0.084 0 rpy=1.5708 0 0 -> xyz=0 -0.09415 0 rpy=1.5708 0 0
- joint joint6output_to_joint6: origin xyz=0 0.06635 0 rpy=-1.5708 0 0 -> xyz=0 0.055 0 rpy=-1.5708 0 0

File: mycobot_description/urdf/new_320_urdf/new_mycobot_pro_320_gripper.urdf (robot description, URDF)
Before this commit: robot firefighter, 14 links, 13 joints
Joints:
- joint joint2_to_joint1: origin xyz=0 0 0.162 rpy=0 0 0 -> xyz=0 0 0.173 rpy=0 0 0
- joint joint3_to_joint2: origin xyz=0 0 0 rpy=0 -1.5708 1.5708 -> xyz=0 -0.086 0 rpy=0 -1.5708 1.5708
- joint joint4_to_joint3: origin xyz=0.13635 0 0    rpy=0 0 0 -> xyz=0.13635 0 -0.086    rpy=0 0 0
- joint joint5_to_joint4: origin xyz=0.1205 0 0.082  rpy= 0 0 1.57080 -> xyz=0.1195 0 0.082  rpy= 0 0 1.57080
- joint joint6_to_joint5: origin xyz=0 -0.084 0.0 rpy=1.5708 0 0 -> xyz=0 -0.09415 0.0 rpy=1.5708 0 0
- joint joint6output_to_joint6: origin xyz=0 0.06635 0.0 rpy=-1.5708 0 0 -> xyz=0 0.055 0.0 rpy=-1.5708 0 0
