Commit message: fix cobotx_b450 urdf model

File: mycobot_description/urdf/cobotx_b450/cobotx_b450.urdf (robot description, URDF)
Before this commit: robot firefighter, 18 links, 17 joints
Joints:
- joint body: limit lower=-3.14 upper=3.14159 effort=1000.0 velocity=0 -> lower=-2.0594 upper=2.0594 effort=1000.0 velocity=0
- joint eye: limit lower=0 upper=0.7853 effort=1000.0 velocity=0 -> lower=0 upper=0.8377 effort=1000.0 velocity=0
- joint head: limit lower=-3.14 upper=3.14159 effort=1000.0 velocity=0 -> lower=-2.4085 upper=3.2812 effort=1000.0 velocity=0
- joint joint1_L: limit lower=-2.8797 upper=2.8797 effort=1000.0 velocity=0 -> lower=-3.1066 upper=3.1066 effort=1000.0 velocity=0
- joint joint1_R: limit lower=-2.8797 upper=2.8797 effort=1000.0 velocity=0 -> lower=-3.1066 upper=3.1066 effort=1000.0 velocity=0
- joint joint2_L: limit lower=-1.7453 upper=1.7453 effort=1000.0 velocity=0 -> lower=-1.4311 upper=2.2689 effort=1000.0 velocity=0; origin xyz= 0 0 0.0   rpy=-1.5708 0 0 -> xyz= 0 0 0   rpy=-1.5708 0 0
- joint joint2_R: limit lower=-1.7453 upper=1.7453 effort=1000.0 velocity=0 -> lower=-1.4311 upper=2.2689 effort=1000.0 velocity=0; origin xyz= 0 0 0.0   rpy=-1.5708 0 0 -> xyz= 0 0 0   rpy=-1.5708 0 0
- joint joint3_L: limit lower=-2.8797 upper=2.8797 effort=1000.0 velocity=0 -> lower=-3.1066 upper=3.1066 effort=1000.0 velocity=0; origin xyz= 0 -0.11 0.0   rpy=1.5708 0 0 -> xyz= 0 -0.11 0   rpy=1.5708 0 0
- joint joint3_R: limit lower=-2.8797 upper=2.8797 effort=1000.0 velocity=0 -> lower=-3.1066 upper=3.1066 effort=1000.0 velocity=0; origin xyz= 0 -0.11 0.0   rpy=1.5708 0 0 -> xyz= 0 -0.11 0   rpy=1.5708 0 0
- joint joint4_L: limit lower=-3.0543 upper=0.0174 effort=1000.0 velocity=0 -> lower=-3.0543 upper=0.2617 effort=1000.0 velocity=0
- joint joint4_R: limit lower=-3.0543 upper=0.0174 effort=1000.0 velocity=0 -> lower=-3.0543 upper=0.2617 effort=1000.0 velocity=0
- joint joint5_L: limit lower=-2.8797 upper=2.8797 effort=1000.0 velocity=0 -> lower=-3.1066 upper=3.1066 effort=1000.0 velocity=0
- joint joint5_R: limit lower=-2.8797 upper=2.8797 effort=1000.0 velocity=0 -> lower=-3.1066 upper=3.1066 effort=1000.0 velocity=0
- joint joint6_L: limit lower=-0.0174 upper=3.14159 effort=1000.0 velocity=0 -> lower=-0.0174 upper=2.9321 effort=1000.0 velocity=0; origin xyz= 0 0.0 0.08 rpy=1.5708 0 0 -> xyz= 0 0 0.08 rpy=1.5708 0 0
- joint joint6_R: limit lower=-0.0174 upper=3.14159 effort=1000.0 velocity=0 -> lower=-0.0174 upper=2.9321 effort=1000.0 velocity=0; origin xyz= 0 0.0 0.08 rpy=1.5708 0 0 -> xyz= 0 0 0.08 rpy=1.5708 0 0
- joint joint7_L: limit lower=-2.8797 upper=2.8797 effort=1000.0 velocity=0 -> lower=-3.1066 upper=3.1066 effort=1000.0 velocity=0
- joint joint7_R: limit lower=-2.8797 upper=2.8797 effort=1000.0 velocity=0 -> lower=-3.1066 upper=3.1066 effort=1000.0 velocity=0

Commit message: add ROS1 cobotx_b450_moveit function frame

File: mycobot_description/urdf/cobotx_b450/cobotx_b450.urdf (robot description, URDF)
Before this commit: robot firefighter, 18 links, 17 joints
Joints:
- joint body: origin xyz= 0 0 0.22    rpy=0 0 0 -> xyz= 0 0 0.231    rpy=0 0 0
