Commit message: add mercury A1、B1 gazebo model in ubuntu 18.04 ros1 melodic

File: Mercury/mercury_b1_moveit/config/gazebo_mercury_b1.urdf (robot description, URDF)
Before this commit: robot firefighter, 18 links, 17 joints
Links:
- added link base_footprint
- link base: mass 0.1 -> 100
Joints:
- added joint base_footprint_joint: type fixed, parent base_footprint, child base
- joint body: origin xyz= 0 0 0.22    rpy=0 0 0 -> xyz= 0 0 0.231    rpy=0 0 0
