Commit message: update mercury urdf joint range

File: mycobot_description/urdf/mercury_a1/mercury_a1.urdf (robot description, URDF)
Before this commit: robot firefighter, 8 links, 7 joints
Joints:
- joint joint1_to_base: limit lower=-2.8797 upper=2.8797 effort=1000.0 velocity=0 -> lower=-3.1066 upper=3.1066 effort=1000.0 velocity=0
- joint joint2_to_joint1: limit lower=-1.7453 upper=1.7453 effort=1000.0 velocity=0 -> lower=-1.4311 upper=2.2689 effort=1000.0 velocity=0
- joint joint3_to_joint2: limit lower=-2.8797 upper=2.8797 effort=1000.0 velocity=0 -> lower=-3.1066 upper=3.1066 effort=1000.0 velocity=0
- joint joint4_to_joint3: limit lower=-3.0543 upper=0.0174 effort=1000.0 velocity=0 -> lower=-3.0543 upper=0.2617 effort=1000.0 velocity=0
- joint joint5_to_joint4: limit lower=-2.8797 upper=2.8797 effort=1000.0 velocity=0 -> lower=-3.1066 upper=3.1066 effort=1000.0 velocity=0
- joint joint6_to_joint5: limit lower=-0.0174 upper=3.14159 effort=1000.0 velocity=0 -> lower=-0.0349 upper=2.9321 effort=1000.0 velocity=0
- joint joint7_to_joint6: limit lower=-2.8797 upper=2.8797 effort=1000.0 velocity=0 -> lower=-3.1066 upper=3.1066 effort=1000.0 velocity=0

File: mycobot_description/urdf/mercury_b1/mercury_b1.urdf (robot description, URDF)
Before this commit: robot firefighter, 18 links, 17 joints
Joints:
- joint eye: origin xyz= 0.03 0 -0.08    rpy=1.5708 0 0 -> xyz= 0.03 0 -0.08    rpy=1.5708 0 3.14
- joint joint6_L: limit lower=-0.0174 upper=2.9321 effort=1000.0 velocity=0 -> lower=-0.0349 upper=2.9321 effort=1000.0 velocity=0
- joint joint6_R: limit lower=-0.0174 upper=2.9321 effort=1000.0 velocity=0 -> lower=-0.0349 upper=2.9321 effort=1000.0 velocity=0
