Commit message: update mercury ros

File: mycobot_description/urdf/mercury_b1/mercury_b1.urdf (robot description, URDF)
Before this commit: robot firefighter, 18 links, 17 joints
Joints:
- joint eye: limit lower=0 upper=0.8377 effort=1000.0 velocity=0 -> lower=0 upper=0.83 effort=1000.0 velocity=0; origin xyz= 0.03 0 -0.08    rpy=1.5708 0 3.14 -> xyz= 0.03 0 -0.08    rpy=1.5708 0 0
