Commit message: update 280 Jetson Nano URDF

File: mycobot_description/urdf/280jn/mycobot_urdf.urdf (robot description, URDF)
Before this commit: robot firefighter, 7 links, 6 joints
Links:
- link joint1: geometry collision mesh filename=package://mycobot_description/urdf/280jn/joint1_jet.dae; visual mesh filename=package://mycobot_description/urdf/280jn/joint1_jet.dae
- link joint2: geometry collision mesh filename=package://mycobot_description/urdf/280jn/joint2.dae; visual mesh filename=package://mycobot_description/urdf/280jn/joint2.dae
- link joint3: geometry collision mesh filename=package://mycobot_description/urdf/280jn/joint3.dae; visual mesh filename=package://mycobot_description/urdf/280jn/joint3.dae
- link joint4: geometry collision mesh filename=package://mycobot_description/urdf/280jn/joint4.dae; visual mesh filename=package://mycobot_description/urdf/280jn/joint4.dae
- link joint5: geometry collision mesh filename=package://mycobot_description/urdf/280jn/joint5.dae; visual mesh filename=package://mycobot_description/urdf/280jn/joint5.dae
- link joint6: geometry collision mesh filename=package://mycobot_description/urdf/280jn/joint6.dae; visual mesh filename=package://mycobot_description/urdf/280jn/joint6.dae
- link joint6_flange: geometry collision mesh filename=package://mycobot_description/urdf/280jn/joint7.dae; visual mesh filename=package://mycobot_description/urdf/280jn/joint7.dae
