Commit message: add flange_camera.urdf

File: mycobot_description/urdf/mycobot_pro_630/my630.urdf (robot description, URDF)
Before this commit: robot firefighter, 4 links, 3 joints
Links:
- added link joint4; collision mesh filename=package://mycobot_description/urdf/mycobot_pro_630/J5-W.dae; visual mesh filename=package://mycobot_description/urdf/mycobot_pro_630/J5-W.dae
- added link joint5; collision mesh filename=package://mycobot_description/urdf/mycobot_pro_630/J6W.dae; visual mesh filename=package://mycobot_description/urdf/mycobot_pro_630/J6W.dae
- added link joint6; collision mesh filename=package://mycobot_description/urdf/mycobot_pro_630/J6-W.dae; visual mesh filename=package://mycobot_description/urdf/mycobot_pro_630/J6-W.dae
- link base: geometry collision mesh filename=package://mycobot_description/urdf/mycobot_pro_630/J1-W.dae; visual mesh filename=package://mycobot_description/urdf/mycobot_pro_630/J1-W.dae
- link joint1: geometry collision mesh filename=package://mycobot_description/urdf/mycobot_pro_630/J2-W.dae; visual mesh filename=package://mycobot_description/urdf/mycobot_pro_630/J2-W.dae
- link joint2: geometry collision mesh filename=package://mycobot_description/urdf/mycobot_pro_630/J3-W.dae; visual mesh filename=package://mycobot_description/urdf/mycobot_pro_630/J3-W.dae
- link joint3: geometry collision mesh filename=package://mycobot_description/urdf/mycobot_pro_630/J4-W.dae; visual mesh filename=package://mycobot_description/urdf/mycobot_pro_630/J4-W.dae
Joints:
- added joint joint4_to_joint3: type revolute, parent joint3, child joint4, origin xyz=0 0.25 -0.03    rpy=0 0 0, axis  0 0 1, limit lower=-3.14 upper=3.14 effort=1000.0 velocity=0
- added joint joint5_to_joint4: type revolute, parent joint4, child joint5, origin xyz=0 0.055 0.055 rpy=1.5707 -1.5707 0, axis 0 0 -1, limit lower=-2.99 upper=2.99 effort=1000.0 velocity=0
- added joint joint6_to_joint5: type revolute, parent joint5, child joint6, origin xyz=0.0495 0 -0.0405 rpy=-1.5707 0 -1.5706 , axis 0 0 1, limit lower=-3.03 upper=3.0368 effort=1000.0 velocity=0
- joint joint1_to_base: origin xyz=0 0 0.16034 rpy=0 0 0 -> xyz=0 0 0.156 rpy=0 0 0
- joint joint2_to_joint1: axis 0 0 -1 -> 0 0 1; limit lower=-2.26 upper=2.26 effort=1000.0 velocity=0 -> lower=-3.14 upper=3.14 effort=1000.0 velocity=0; origin xyz=0 -0.035  0.09 rpy=1.5707 0 0 -> xyz=0 0.05  0.083  rpy=1.5707 0 3.14159
- joint joint3_to_joint2: axis  0 0 -1 ->  0 0 1; limit lower=-2.61 upper=2.618 effort=1000.0 velocity=0 -> lower=-3.14 upper=3.14 effort=1000.0 velocity=0
