Commit message: 增加320力控夹爪滑块控制、320PI增加pro自适应夹爪

File: mycobot_description/urdf/force_control_gripper/mycobot_pro_force_gripper.urdf (robot description, URDF)
Before this commit: robot firefighter1, 1 links, 0 joints
Links:
- added link gripper_left1; collision mesh filename=package://mycobot_description/urdf/force_control_gripper/pr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; visual mesh filename=package://mycobot_description/urdf/force_control_gripper/pr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
- added link gripper_left2; collision mesh filename=package://mycobot_description/urdf/force_control_gripper/pr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; visual mesh filename=package://mycobot_description/urdf/force_control_gripper/pr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
- added link gripper_left3; collision mesh filename=package://mycobot_description/urdf/force_control_gripper/pr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; visual mesh filename=package://mycobot_description/urdf/force_control_gripper/pr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
- added link gripper_right1; collision mesh filename=package://mycobot_description/urdf/force_control_gripper/pr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; visual mesh filename=package://mycobot_description/urdf/force_control_gripper/pr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
- added link gripper_right2; collision mesh filename=package://mycobot_description/urdf/force_control_gripper/pr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; visual mesh filename=package://mycobot_description/urdf/force_control_gripper/pr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
- added link gripper_right3; collision mesh filename=package://mycobot_description/urdf/force_control_gripper/pr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; visual mesh filename=package://mycobot_description/urdf/force_control_gripper/pr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
- link gripper_base: geometry collision mesh filename=package://mycobot_description/urdf/force_control_gripper/pr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; visual mesh filename=package://mycobot_description/urdf/force_control_gripper/pr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
Joints:
- added joint gripper_base_to_gripper_left2: type revolute, parent gripper_base, child gripper_left2, origin xyz=-0.0445 -0.004 -0.02 rpy=0 0 0, axis 0 0 1, limit lower=-0.8 upper=0.5 effort=1000.0 velocity=0, mimic joint=gripper_controller multiplier=1.0 offset=0
- added joint gripper_base_to_gripper_right2: type revolute, parent gripper_base, child gripper_right2, origin xyz=0.0442 -0.004 -0.02 rpy=0 0 0, axis 0 0 1, limit lower=-0.5 upper=0.8 effort=1000.0 velocity=0, mimic joint=gripper_controller multiplier=-1.0 offset=0
- added joint gripper_base_to_gripper_right3: type revolute, parent gripper_base, child gripper_right3, origin xyz=0.018 0.015 -0.0212 rpy=0 0 0, axis 0 0 1, limit lower=1 upper=0 effort=1000.0 velocity=0, mimic joint=gripper_controller multiplier=-1.0 offset=0
- added joint gripper_controller: type revolute, parent gripper_base, child gripper_left3, origin xyz=-0.018 0.016 -0.02 rpy=0 0 0, axis 0 0 1, limit lower=0 upper=1 effort=1000.0 velocity=0
- added joint gripper_left3_to_gripper_left1: type revolute, parent gripper_left3, child gripper_left1, origin xyz=0.01 0.06 0.0 rpy=0 0 0, axis 0 0 1, limit lower=-0.5 upper=0.5 effort=1000.0 velocity=0, mimic joint=gripper_controller multiplier=-1.0 offset=0
- added joint gripper_right3_to_gripper_right1: type revolute, parent gripper_right3, child gripper_right1, origin xyz=-0.01 0.061 0.001 rpy=0 0 0, axis 0 0 1, limit lower=-0.5 upper=0.5 effort=1000.0 velocity=0, mimic joint=gripper_controller multiplier=1.0 offset=0

File: mycobot_description/urdf/mycobot_320_m5_2022/new_mycobot_pro_320_m5_2022_gripper.urdf (robot description, URDF)
Before this commit: robot firefighter, 14 links, 13 joints
Joints:
- joint joint2_to_joint1: limit lower=-2.96 upper=2.96 effort=1000.0 velocity=0 -> lower=-2.93 upper=2.93 effort=1000.0 velocity=0
- joint joint3_to_joint2: limit lower=-2.79 upper=2.79 effort=1000.0 velocity=0 -> lower=-2.35 upper=2.35 effort=1000.0 velocity=0
- joint joint4_to_joint3: limit lower=-2.79 upper=2.79 effort=1000.0 velocity=0 -> lower=-2.53 upper=2.53 effort=1000.0 velocity=0
- joint joint5_to_joint4: limit lower=-2.79 upper=2.79 effort=1000.0 velocity=0 -> lower=-2.58 upper=2.58 effort=1000.0 velocity=0
- joint joint6_to_joint5: limit lower=-2.96 upper=2.96 effort=1000.0 velocity=0 -> lower=-2.93 upper=2.93 effort=1000.0 velocity=0
- joint joint6output_to_joint6: limit lower=-3.05 upper=3.05 effort=1000.0 velocity=0 -> lower=-3.14 upper=3.14 effort=1000.0 velocity=0
