Commit message: 320M5/PI增加力控夹爪ros1 moveit、320PI版本增加Pro自适应夹爪demo

File: mycobot_description/urdf/mycobot_320_m5_2022/new_mycobot_pro_320_m5_2022_gripper.urdf (robot description, URDF)
Before this commit: robot firefighter, 14 links, 13 joints
Joints:
- joint joint6output_to_gripper_base: origin xyz=0 0.0 0.034 rpy=1.5708 0 0 -> xyz=0 0.0 0.042 rpy=1.5708 0 0
