Commit message: 320力控夹爪URDF增加细节零件

File: mycobot_description/urdf/mycobot_320_m5_2022/pro_320_m5_2022_force_gripper.urdf (robot description, URDF)
Before this commit: robot firefighter, 15 links, 14 joints
Joints:
- joint joint6output_to_gripper_base: origin xyz=0 -0.02 0.036 rpy=1.5708 0 0 -> xyz=0 -0.02 0.0364 rpy=1.5708 0 0

File: mycobot_description/urdf/mycobot_320_m5_2022/pro_320_m5_2022_moveit_force_gripper.urdf (robot description, URDF)
Before this commit: robot firefighter, 15 links, 14 joints
Joints:
- joint joint6output_to_gripper_base: origin xyz=0 -0.02 0.036 rpy=1.5708 0 0 -> xyz=0 -0.02 0.0364 rpy=1.5708 0 0

File: mycobot_description/urdf/mycobot_320_pi_2022/pro_320_pi_2022_force_gripper.urdf (robot description, URDF)
Before this commit: robot firefighter, 15 links, 14 joints
Joints:
- joint joint6output_to_gripper_base: origin xyz=0 -0.02 0.036 rpy=1.5708 0 0 -> xyz=0 -0.02 0.0364 rpy=1.5708 0 0

File: mycobot_description/urdf/mycobot_320_pi_2022/pro_320_pi_2022_moveit_force_gripper.urdf (robot description, URDF)
Before this commit: robot firefighter, 15 links, 14 joints
Joints:
- joint joint6output_to_gripper_base: origin xyz=0 -0.02 0.036 rpy=1.5708 0 0 -> xyz=0 -0.02 0.0364 rpy=1.5708 0 0
