Commit message: update 320 URDF args

File: mycobot_description/urdf/mycobot_320_m5_2022/new_mycobot_pro_320_m5_2022.urdf (robot description, URDF)
Before this commit: robot firefighter, 7 links, 6 joints
Joints:
- joint joint2_to_joint1: origin xyz=0 0 0.173 rpy=0 0 0 -> xyz=0 0 0.1739 rpy=0 0 0
- joint joint3_to_joint2: origin xyz=0 -0.086 0 rpy=0 -1.5708 1.5708 -> xyz=0 -0.08878 0 rpy=0 -1.5708 1.5708
- joint joint4_to_joint3: origin xyz=0.13635 0 -0.086    rpy=0 0 0 -> xyz=0.135 0 -0.08878    rpy=0 0 0
- joint joint5_to_joint4: origin xyz=0.1195 0 0.082  rpy= 0 0 1.57080 -> xyz=0.120 0 0.08878  rpy= 0 0 1.57080
- joint joint6_to_joint5: origin xyz=0 -0.09415 0.0 rpy=1.5708 0 0 -> xyz=0 -0.095 0.0 rpy=1.5708 0 0
- joint joint6output_to_joint6: origin xyz=0 0.055 0.0 rpy=-1.5708 0 0 -> xyz=0 0.0655 0.0 rpy=-1.5708 0 0

File: mycobot_description/urdf/mycobot_320_m5_2022/new_mycobot_pro_320_m5_2022_gripper.urdf (robot description, URDF)
Before this commit: robot firefighter, 14 links, 13 joints
Joints:
- joint joint2_to_joint1: origin xyz=0 0 0.173 rpy=0 0 0 -> xyz=0 0 0.1739 rpy=0 0 0
- joint joint3_to_joint2: origin xyz=0 -0.086 0 rpy=0 -1.5708 1.5708 -> xyz=0 -0.08878 0 rpy=0 -1.5708 1.5708
- joint joint4_to_joint3: origin xyz=0.13635 0 -0.086    rpy=0 0 0 -> xyz=0.135 0 -0.08878    rpy=0 0 0
- joint joint5_to_joint4: origin xyz=0.1195 0 0.082  rpy= 0 0 1.57080 -> xyz=0.120 0 0.08878  rpy= 0 0 1.57080
- joint joint6_to_joint5: origin xyz=0 -0.09415 0.0 rpy=1.5708 0 0 -> xyz=0 -0.095 0.0 rpy=1.5708 0 0
- joint joint6output_to_joint6: origin xyz=0 0.055 0.0 rpy=-1.5708 0 0 -> xyz=0 0.0655 0.0 rpy=-1.5708 0 0

File: mycobot_description/urdf/mycobot_320_m5_2022/new_mycobot_pro_320_m5_2022_moveit_gripper.urdf (robot description, URDF)
Before this commit: robot firefighter, 14 links, 13 joints
Joints:
- joint joint2_to_joint1: origin xyz=0 0 0.173 rpy=0 0 0 -> xyz=0 0 0.1739 rpy=0 0 0
- joint joint3_to_joint2: origin xyz=0 -0.086 0 rpy=0 -1.5708 1.5708 -> xyz=0 -0.08878 0 rpy=0 -1.5708 1.5708
- joint joint4_to_joint3: origin xyz=0.13635 0 -0.086    rpy=0 0 0 -> xyz=0.135 0 -0.08878    rpy=0 0 0
- joint joint5_to_joint4: origin xyz=0.1195 0 0.082  rpy= 0 0 1.57080 -> xyz=0.120 0 0.08878  rpy= 0 0 1.57080
- joint joint6_to_joint5: origin xyz=0 -0.09415 0.0 rpy=1.5708 0 0 -> xyz=0 -0.095 0.0 rpy=1.5708 0 0
- joint joint6output_to_joint6: origin xyz=0 0.055 0.0 rpy=-1.5708 0 0 -> xyz=0 0.0655 0.0 rpy=-1.5708 0 0

File: mycobot_description/urdf/mycobot_320_m5_2022/new_mycobot_pro_320moveit_m5_2022.urdf (robot description, URDF)
Before this commit: robot firefighter, 7 links, 6 joints
Joints:
- joint joint2_to_joint1: origin xyz=0 0 0.173 rpy=0 0 0 -> xyz=0 0 0.1739 rpy=0 0 0
- joint joint3_to_joint2: origin xyz=0 -0.086 0 rpy=0 -1.57080  1.57080 -> xyz=0 -0.08878 0 rpy=0 -1.57080  1.57080
- joint joint4_to_joint3: origin xyz=0.13635 0 -0.086    rpy=0 0 0 -> xyz=0.135 0 -0.08878    rpy=0 0 0
- joint joint5_to_joint4: origin xyz=0.1195 0  0.082 rpy=0 0 1.57080 -> xyz=0.120 0  0.08878 rpy=0 0 1.57080
- joint joint6_to_joint5: origin xyz=0 -0.09415 0 rpy=1.57080 0 0 -> xyz=0 -0.095 0 rpy=1.57080 0 0
- joint joint6output_to_joint6: origin xyz=0 0.055 0 rpy=-1.57080 0 0  -> xyz=0 0.0655 0 rpy=-1.57080 0 0 

File: mycobot_description/urdf/mycobot_320_m5_2022/pro_320_m5_2022_force_gripper.urdf (robot description, URDF)
Before this commit: robot firefighter, 15 links, 14 joints
Joints:
- joint joint2_to_joint1: origin xyz=0 0 0.173 rpy=0 0 0 -> xyz=0 0 0.1739 rpy=0 0 0
- joint joint3_to_joint2: origin xyz=0 -0.086 0 rpy=0 -1.5708 1.5708 -> xyz=0 -0.08878 0 rpy=0 -1.5708 1.5708
- joint joint4_to_joint3: origin xyz=0.13635 0 -0.086    rpy=0 0 0 -> xyz=0.135 0 -0.08878    rpy=0 0 0
- joint joint5_to_joint4: origin xyz=0.1195 0 0.082  rpy= 0 0 1.57080 -> xyz=0.120 0 0.08878  rpy= 0 0 1.57080
- joint joint6_to_joint5: origin xyz=0 -0.09415 0.0 rpy=1.5708 0 0 -> xyz=0 -0.095 0.0 rpy=1.5708 0 0
- joint joint6output_to_joint6: origin xyz=0 0.055 0.0 rpy=-1.5708 0 0 -> xyz=0 0.0655 0.0 rpy=-1.5708 0 0

File: mycobot_description/urdf/mycobot_320_m5_2022/pro_320_m5_2022_moveit_force_gripper.urdf (robot description, URDF)
Before this commit: robot firefighter, 15 links, 14 joints
Joints:
- joint joint2_to_joint1: origin xyz=0 0 0.173 rpy=0 0 0 -> xyz=0 0 0.1739 rpy=0 0 0
- joint joint3_to_joint2: origin xyz=0 -0.086 0 rpy=0 -1.5708 1.5708 -> xyz=0 -0.08878 0 rpy=0 -1.5708 1.5708
- joint joint4_to_joint3: origin xyz=0.13635 0 -0.086    rpy=0 0 0 -> xyz=0.135 0 -0.08878    rpy=0 0 0
- joint joint5_to_joint4: origin xyz=0.1195 0 0.082  rpy= 0 0 1.57080 -> xyz=0.120 0 0.08878  rpy= 0 0 1.57080
- joint joint6_to_joint5: origin xyz=0 -0.09415 0.0 rpy=1.5708 0 0 -> xyz=0 -0.095 0.0 rpy=1.5708 0 0
- joint joint6output_to_joint6: origin xyz=0 0.055 0.0 rpy=-1.5708 0 0 -> xyz=0 0.0655 0.0 rpy=-1.5708 0 0

File: mycobot_description/urdf/mycobot_320_m5_2022/pro_320_m5_2022_moveit_three_gripper.urdf (robot description, URDF)
Before this commit: robot firefighter, 8 links, 7 joints
Joints:
- joint joint2_to_joint1: origin xyz=0 0 0.173 rpy=0 0 0 -> xyz=0 0 0.1739 rpy=0 0 0
- joint joint3_to_joint2: origin xyz=0 -0.086 0 rpy=0 -1.57080  1.57080 -> xyz=0 -0.08878 0 rpy=0 -1.57080  1.57080
- joint joint4_to_joint3: origin xyz=0.13635 0 -0.086    rpy=0 0 0 -> xyz=0.135 0 -0.08878    rpy=0 0 0
- joint joint5_to_joint4: origin xyz=0.1195 0  0.082 rpy=0 0 1.57080 -> xyz=0.120 0  0.08878 rpy=0 0 1.57080
- joint joint6_to_joint5: origin xyz=0 -0.09415 0 rpy=1.57080 0 0 -> xyz=0 -0.095 0 rpy=1.57080 0 0
- joint joint6output_to_joint6: origin xyz=0 0.055 0 rpy=-1.57080 0 0  -> xyz=0 0.0655 0 rpy=-1.57080 0 0 

File: mycobot_description/urdf/mycobot_320_pi_2022/new_mycobot_pro_320_pi_2022.urdf (robot description, URDF)
Before this commit: robot firefighter, 7 links, 6 joints
Joints:
- joint joint2_to_joint1: origin xyz=0 0 0.173 rpy=0 0 0 -> xyz=0 0 0.1739 rpy=0 0 0
- joint joint3_to_joint2: origin xyz=0 -0.086 0 rpy=0 -1.5708 1.5708 -> xyz=0 -0.08878 0 rpy=0 -1.5708 1.5708
- joint joint4_to_joint3: origin xyz=0.13635 0 -0.086    rpy=0 0 0 -> xyz=0.135 0 -0.08878    rpy=0 0 0
- joint joint5_to_joint4: origin xyz=0.1195 0 0.082  rpy= 0 0 1.57080 -> xyz=0.120 0 0.08878  rpy= 0 0 1.57080
- joint joint6_to_joint5: origin xyz=0 -0.09415 0 rpy=1.5708 0 0 -> xyz=0 -0.095 0 rpy=1.5708 0 0
- joint joint6output_to_joint6: origin xyz=0 0.06635 0 rpy=-1.5708 0 0 -> xyz=0 0.0655 0 rpy=-1.5708 0 0

File: mycobot_description/urdf/mycobot_320_pi_2022/new_mycobot_pro_320_pi_2022_gripper.urdf (robot description, URDF)
Before this commit: robot firefighter, 14 links, 13 joints
Joints:
- joint joint2_to_joint1: origin xyz=0 0 0.173 rpy=0 0 0 -> xyz=0 0 0.1739 rpy=0 0 0
- joint joint3_to_joint2: origin xyz=0 -0.086 0 rpy=0 -1.5708 1.5708 -> xyz=0 -0.08878 0 rpy=0 -1.5708 1.5708
- joint joint4_to_joint3: origin xyz=0.13635 0 -0.086    rpy=0 0 0 -> xyz=0.135 0 -0.08878    rpy=0 0 0
- joint joint5_to_joint4: origin xyz=0.1195 0 0.082  rpy= 0 0 1.57080 -> xyz=0.120 0 0.08878  rpy= 0 0 1.57080
- joint joint6_to_joint5: origin xyz=0 -0.09415 0.0 rpy=1.5708 0 0 -> xyz=0 -0.095 0.0 rpy=1.5708 0 0
- joint joint6output_to_joint6: origin xyz=0 0.055 0.0 rpy=-1.5708 0 0 -> xyz=0 0.0655 0.0 rpy=-1.5708 0 0

File: mycobot_description/urdf/mycobot_320_pi_2022/new_mycobot_pro_320_pi_2022_moveit_gripper.urdf (robot description, URDF)
Before this commit: robot firefighter, 14 links, 13 joints
Joints:
- joint joint2_to_joint1: origin xyz=0 0 0.173 rpy=0 0 0 -> xyz=0 0 0.1739 rpy=0 0 0
- joint joint3_to_joint2: origin xyz=0 -0.086 0 rpy=0 -1.5708 1.5708 -> xyz=0 -0.08878 0 rpy=0 -1.5708 1.5708
- joint joint4_to_joint3: origin xyz=0.13635 0 -0.086    rpy=0 0 0 -> xyz=0.135 0 -0.08878    rpy=0 0 0
- joint joint5_to_joint4: origin xyz=0.1195 0 0.082  rpy= 0 0 1.57080 -> xyz=0.120 0 0.08878  rpy= 0 0 1.57080
- joint joint6_to_joint5: origin xyz=0 -0.09415 0.0 rpy=1.5708 0 0 -> xyz=0 -0.095 0.0 rpy=1.5708 0 0
- joint joint6output_to_joint6: origin xyz=0 0.055 0.0 rpy=-1.5708 0 0 -> xyz=0 0.0655 0.0 rpy=-1.5708 0 0

File: mycobot_description/urdf/mycobot_320_pi_2022/new_mycobot_pro_320_pi_moveit_2022.urdf (robot description, URDF)
Before this commit: robot firefighter, 7 links, 6 joints
Joints:
- joint joint2_to_joint1: origin xyz=0 0 0.173 rpy=0 0 0 -> xyz=0 0 0.1739 rpy=0 0 0
- joint joint3_to_joint2: origin xyz=0 -0.086  0 rpy=0 -1.57080  1.57080 -> xyz=0 -0.08878  0 rpy=0 -1.57080  1.57080
- joint joint4_to_joint3: origin xyz=0.13635 0 -0.086    rpy=0 0 0 -> xyz=0.135 0 -0.08878   rpy=0 0 0
- joint joint5_to_joint4: origin xyz=0.1195 0  0.082 rpy=0 0 1.57080 -> xyz=0.120  0.08878 rpy=0 0 1.57080
- joint joint6_to_joint5: origin xyz=0 -0.09415 0 rpy=1.57080 0 0 -> xyz=0 -0.095 0 rpy=1.57080 0 0
- joint joint6output_to_joint6: origin xyz=0 0.055 0 rpy=-1.57080 0 0  -> xyz=0 0.0655 0 rpy=-1.57080 0 0 

File: mycobot_description/urdf/mycobot_320_pi_2022/new_mycobot_vision_v2_2022.urdf (robot description, URDF)
Before this commit: robot firefighter, 8 links, 7 joints
Joints:
- joint joint2_to_joint1: origin xyz=0 0 0.173 rpy=0 0 0 -> xyz=0 0 0.1739 rpy=0 0 0
- joint joint3_to_joint2: origin xyz=0 -0.086 0 rpy=0 -1.5708 1.5708 -> xyz=0 -0.08878 0 rpy=0 -1.5708 1.5708
- joint joint4_to_joint3: origin xyz=0.13635 0 -0.086    rpy=0 0 0 -> xyz=0.135 0 -0.08878    rpy=0 0 0
- joint joint5_to_joint4: origin xyz=0.1195 0 0.082  rpy= 0 0 1.57080 -> xyz=0.120 0 0.08878  rpy= 0 0 1.57080
- joint joint6_to_joint5: origin xyz=0 -0.09415 0 rpy=1.5708 0 0 -> xyz=0 -0.095 0 rpy=1.5708 0 0
- joint joint6output_to_joint6: origin xyz=0 0.055 0 rpy=-1.5708 0 0 -> xyz=0 0.0655 0 rpy=-1.5708 0 0

File: mycobot_description/urdf/mycobot_320_pi_2022/pro_320_pi_2022_force_gripper.urdf (robot description, URDF)
Before this commit: robot firefighter, 15 links, 14 joints
Joints:
- joint joint2_to_joint1: origin xyz=0 0 0.173 rpy=0 0 0 -> xyz=0 0 0.1739 rpy=0 0 0
- joint joint3_to_joint2: origin xyz=0 -0.086 0 rpy=0 -1.5708 1.5708 -> xyz=0 -0.08878 0 rpy=0 -1.5708 1.5708
- joint joint4_to_joint3: origin xyz=0.13635 0 -0.086    rpy=0 0 0 -> xyz=0.135 0 -0.08878    rpy=0 0 0
- joint joint5_to_joint4: origin xyz=0.1195 0 0.082  rpy= 0 0 1.57080 -> xyz=0.120 0 0.08878  rpy= 0 0 1.57080
- joint joint6_to_joint5: origin xyz=0 -0.09415 0.0 rpy=1.5708 0 0 -> xyz=0 -0.095 0.0 rpy=1.5708 0 0
- joint joint6output_to_joint6: origin xyz=0 0.06635 0.0 rpy=-1.5708 0 0 -> xyz=0 0.0655 0.0 rpy=-1.5708 0 0

File: mycobot_description/urdf/mycobot_320_pi_2022/pro_320_pi_2022_moveit_force_gripper.urdf (robot description, URDF)
Before this commit: robot firefighter, 15 links, 14 joints
Joints:
- joint joint2_to_joint1: origin xyz=0 0 0.173 rpy=0 0 0 -> xyz=0 0 0.1739 rpy=0 0 0
- joint joint3_to_joint2: origin xyz=0 -0.086 0 rpy=0 -1.5708 1.5708 -> xyz=0 -0.08878 0 rpy=0 -1.5708 1.5708
- joint joint4_to_joint3: origin xyz=0.13635 0 -0.086    rpy=0 0 0 -> xyz=0.135 0 -0.08878    rpy=0 0 0
- joint joint5_to_joint4: origin xyz=0.1195 0 0.082  rpy= 0 0 1.57080 -> xyz=0.120 0 0.08878  rpy= 0 0 1.57080
- joint joint6_to_joint5: origin xyz=0 -0.09415 0.0 rpy=1.5708 0 0 -> xyz=0 -0.095 0.0 rpy=1.5708 0 0
- joint joint6output_to_joint6: origin xyz=0 0.06635 0.0 rpy=-1.5708 0 0 -> xyz=0 0.0655 0.0 rpy=-1.5708 0 0
