Commit message: 增加280JN自适应夹爪URDF模型

File: mycobot_description/urdf/mycobot_280_jn/mycobot_280_jn.urdf (robot description, URDF)
Before this commit: robot firefighter, 7 links, 6 joints
Links:
- added link g_base; collision mesh filename=package://mycobot_description/urdf/mycobot_280_jn/G_base.dae; visual mesh filename=package://mycobot_description/urdf/mycobot_280_jn/G_base.dae
Joints:
- added joint g_base_to_joint1: type fixed, parent g_base, child joint1, origin xyz=0 0 0 rpy=0 0 0, axis 0 0 0, limit lower=-3.14 upper=3.14159 effort=1000.0 velocity=0
- joint joint2_to_joint1: limit lower=-3.14 upper=3.14159 effort=1000.0 velocity=0 -> lower=-2.9321 upper=2.9321 effort=1000.0 velocity=0
- joint joint3_to_joint2: limit lower=-3.14 upper=3.14159 effort=1000.0 velocity=0 -> lower=-2.0943 upper=2.0943 effort=1000.0 velocity=0
- joint joint4_to_joint3: limit lower=-3.14 upper=3.14159 effort=1000.0 velocity=0 -> lower=-2.6179 upper=2.6179 effort=1000.0 velocity=0
- joint joint5_to_joint4: limit lower=-3.14 upper=3.14159 effort=1000.0 velocity=0 -> lower=-2.5307 upper=2.5307 effort=1000.0 velocity=0
- joint joint6_to_joint5: limit lower=-3.14 upper=3.14159 effort=1000.0 velocity=0 -> lower=-2.8797 upper=2.8797 effort=1000.0 velocity=0

Commit message: 更新260/270/280/myarm/mybuddy/p340 urdf模型关节运动范围

File: mycobot_description/urdf/mycobot_280_jn/mycobot_280_jn.urdf (robot description, URDF)
Before this commit: robot firefighter, 8 links, 7 joints
Joints:
- joint joint3_to_joint2: limit lower=-2.0943 upper=2.0943 effort=1000.0 velocity=0 -> lower=-2.3562 upper=2.3562 effort=1000.0 velocity=0

File: mycobot_description/urdf/mycobot_280_jn/mycobot_280_jn_adaptive_gripper_parallel.urdf (robot description, URDF)
Before this commit: robot firefighter, 15 links, 14 joints
Joints:
- joint joint3_to_joint2: limit lower=-2.0943 upper=2.0943 effort=1000.0 velocity=0 -> lower=-2.3562 upper=2.3562 effort=1000.0 velocity=0

File: mycobot_description/urdf/mycobot_280_jn/mycobot_280_jn_adaptive_gripper_vertical.urdf (robot description, URDF)
Before this commit: robot firefighter, 15 links, 14 joints
Joints:
- joint joint3_to_joint2: limit lower=-2.0943 upper=2.0943 effort=1000.0 velocity=0 -> lower=-2.3562 upper=2.3562 effort=1000.0 velocity=0

File: mycobot_description/urdf/mycobot_280_jn/mycobot_280_jn_camera_flange.urdf (robot description, URDF)
Before this commit: robot firefighter, 9 links, 8 joints
Joints:
- joint joint3_to_joint2: limit lower=-2.0943 upper=2.0943 effort=1000.0 velocity=0 -> lower=-2.3562 upper=2.3562 effort=1000.0 velocity=0

File: mycobot_description/urdf/mycobot_280_jn/mycobot_280_jn_parallel_gripper.urdf (robot description, URDF)
Before this commit: robot firefighter, 11 links, 10 joints
Joints:
- joint joint3_to_joint2: limit lower=-2.0943 upper=2.0943 effort=1000.0 velocity=0 -> lower=-2.3562 upper=2.3562 effort=1000.0 velocity=0

File: mycobot_description/urdf/mycobot_280_m5/mycobot_280_m5.urdf (robot description, URDF)
Before this commit: robot firefighter, 8 links, 7 joints
Joints:
- joint joint2_to_joint1: limit lower=-3.14 upper=3.14159 effort=1000.0 velocity=0 -> lower=-2.9322 upper=2.9322 effort=1000.0 velocity=0
- joint joint3_to_joint2: limit lower=-3.14 upper=3.14159 effort=1000.0 velocity=0 -> lower=-2.3562 upper=2.3562 effort=1000.0 velocity=0
- joint joint4_to_joint3: limit lower=-3.14 upper=3.14159 effort=1000.0 velocity=0 -> lower=-2.618 upper=2.618 effort=1000.0 velocity=0
- joint joint5_to_joint4: limit lower=-3.14 upper=3.14159 effort=1000.0 velocity=0 -> lower=-2.5307 upper=2.5307 effort=1000.0 velocity=0
- joint joint6_to_joint5: limit lower=-3.14 upper=3.14159 effort=1000.0 velocity=0 -> lower=-2.8798 upper=2.8798 effort=1000.0 velocity=0
