Commit message: add ros1 myarm c650 package

File: mycobot_description/urdf/myarm_c650/myarm_c650.urdf (robot description, URDF)
Before this commit: robot firefighter, 7 links, 6 joints
Links:
- removed link joint6
- added link endeffector; collision mesh filename=package://mycobot_description/urdf/myarm_c650/endeffector.d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; visual mesh filename=package://mycobot_description/urdf/myarm_c650/endeffector.d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
Joints:
- removed joint joint6_to_joint5
- added joint endeffector_to_joint5: type revolute, parent joint5, child endeffector, origin xyz=0 0.055 0 rpy=-1.5708 0 0, axis 0 0 1, limit lower=-1.9198 upper=1.9198 effort=1000.0 velocity=0
- joint joint3_to_joint2: origin xyz=0 -0.11 0    rpy=1.5708 0 0 -> xyz=0.0565 -0.296 0    rpy=0 0 0
- joint joint4_to_joint3: origin xyz=0.0 0 0.0 rpy=-1.5708 0 3.14159 -> xyz=0.081 0 0.0 rpy=0 1.5708 0
- joint joint5_to_joint4: origin xyz=0 -0.126 0 rpy=1.5708 0 0 -> xyz=0.0 0.0003 0.2517 rpy=1.5708 0 1.5708

Commit message: add ros1 myarm c650 package

File: mycobot_description/urdf/myarm_c650/myarm_c650.urdf (robot description, URDF)
Before this commit: robot firefighter, 7 links, 6 joints
Joints:
- joint endeffector_to_joint5: origin xyz=0 0.055 0 rpy=-1.5708 0 0 -> xyz=0 -0.045 0 rpy=-1.5708 0 0
- joint joint1_to_base: origin xyz=0 0 0.165 rpy=0 0 0 -> xyz=0 0 0.070 rpy=3.14159 0 0
- joint joint2_to_joint1: origin xyz=0 0  0 rpy=-1.5708 0 0 -> xyz=0 0 -0.080 rpy=1.5708 0 0
- joint joint4_to_joint3: origin xyz=0.081 0 0.0 rpy=0 1.5708 0 -> xyz=0.081 0 0.004 rpy=0 -1.5708 0
- joint joint5_to_joint4: origin xyz=0.0 0.0003 0.2517 rpy=1.5708 0 1.5708 -> xyz=0.0 0.0003 -0.250 rpy=-1.5708 3.14159 -1.5708
