Commit message: improve ros1 myarm-c650 code

File: mycobot_description/urdf/myarm_c650/myarm_c650.urdf (robot description, URDF)
Before this commit: robot firefighter, 7 links, 6 joints
Links:
- removed link endeffector
- removed link joint1
- removed link joint2
- removed link joint3
- removed link joint4
- removed link joint5
- added link gripper; collision mesh filename=package://mycobot_description/urdf/myarm_c650/myarm_c_grip_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; visual mesh filename=package://mycobot_description/urdf/myarm_c650/myarm_c_grip_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
- added link gripper_left; collision mesh filename=package://mycobot_description/urdf/myarm_c650/myarm_c_grip_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; visual mesh filename=package://mycobot_description/urdf/myarm_c650/myarm_c_grip_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
- added link gripper_right; collision mesh filename=package://mycobot_description/urdf/myarm_c650/myarm_c_grip_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; visual mesh filename=package://mycobot_description/urdf/myarm_c650/myarm_c_grip_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
- added link link1; collision mesh filename=package://mycobot_description/urdf/myarm_c650/joint1.dae; visual mesh filename=package://mycobot_description/urdf/myarm_c650/joint1.dae
- added link link2; collision mesh filename=package://mycobot_description/urdf/myarm_c650/joint2.dae; visual mesh filename=package://mycobot_description/urdf/myarm_c650/joint2.dae
- added link link3; collision mesh filename=package://mycobot_description/urdf/myarm_c650/joint3.dae; visual mesh filename=package://mycobot_description/urdf/myarm_c650/joint3.dae
- added link link4; collision mesh filename=package://mycobot_description/urdf/myarm_c650/joint4.dae; visual mesh filename=package://mycobot_description/urdf/myarm_c650/joint4.dae
- added link link5; collision mesh filename=package://mycobot_description/urdf/myarm_c650/joint5.dae; visual mesh filename=package://mycobot_description/urdf/myarm_c650/joint5.dae
- link base: geometry collision mesh filename=package://mycobot_description/urdf/myarm_c650/myarm_basic_b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; visual mesh filename=package://mycobot_description/urdf/myarm_c650/myarm_basic_b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
Joints:
- removed joint endeffector_to_joint5
- removed joint joint1_to_base
- removed joint joint2_to_joint1
- removed joint joint3_to_joint2
- removed joint joint4_to_joint3
- removed joint joint5_to_joint4
- added joint gripper: type prismatic, parent gripper, child gripper_left, origin xyz=-0.030 0 -0.066 rpy=3.14 -1.57 1.57, axis 0 0 1, limit lower=0 upper=0.022 effort=1000.0 velocity=0
- added joint gripper_r: type prismatic, parent gripper, child gripper_right, origin xyz=-0.030 0 -0.066 rpy=3.14 -1.57 1.57, axis 0 0 -1, limit lower=0 upper=0.022 effort=1000.0 velocity=0, mimic joint=gripper multiplier=1.0 offset=0
- added joint joint1: type revolute, parent base, child link1, origin xyz=0 0 0.070 rpy=3.14159 0 0, axis 0 0 1, limit lower=-2.7925 upper=2.7925 effort=1000.0 velocity=0
- added joint joint2: type revolute, parent link1, child link2, origin xyz=0 0 -0.080 rpy=1.5708 0 0, axis 0 0 1, limit lower=-1.3962 upper=1.3962 effort=1000.0 velocity=0
- added joint joint3: type revolute, parent link2, child link3, origin xyz=0.0565 -0.296 0    rpy=0 0 0, axis  0 0 1, limit lower=-1.3962 upper=1.32 effort=1000.0 velocity=0
- added joint joint4: type revolute, parent link3, child link4, origin xyz=0.081 0 0.004 rpy=0 -1.5708 0, axis  0 0 1, limit lower=-1.7453 upper=1.7453 effort=1000.0 velocity=0
- added joint joint5: type revolute, parent link4, child link5, origin xyz=0.0 0.0003 -0.250 rpy=-1.5708 3.14159 -1.5708, axis 0 0 1, limit lower=-1.3962 upper=1.3962 effort=1000.0 velocity=0
- added joint joint6: type revolute, parent link5, child gripper, origin xyz=0 -0.055 0 rpy=-1.5708 0 0, axis 0 0 1, limit lower=-1.9198 upper=1.9198 effort=1000.0 velocity=0

File: mycobot_description/urdf/myarm_c650/myarm_c650.urdf.xacro (robot description, xacro)
@@ -5,5 +5,5 @@
     <visual>
       <geometry>
-       <mesh filename="package://mycobot_description/urdf/myarm_c650/base.dae"/>
+       <mesh filename="package://mycobot_description/urdf/myarm_c650/myarm_basic_base.dae"/>
       </geometry>
       <origin xyz = "0.0 0 0 " rpy = " 0 0 0"/>
@@ -11,10 +11,10 @@
     <collision>
       <geometry>
-       <mesh filename="package://mycobot_description/urdf/myarm_c650/base.dae"/>
+       <mesh filename="package://mycobot_description/urdf/myarm_c650/bamyarm_basic_basese.dae"/>
         </geometry>
         <origin xyz = "0.0 0 0 " rpy = " 0 0 0"/>
     </collision>
   </link>
-  <link name="joint1">
+  <link name="link1">
     <visual>
       <geometry>
@@ -30,5 +30,5 @@
     </collision>
   </link>
-  <link name="joint2">
+  <link name="link2">
     <visual>
       <geometry>
@@ -44,5 +44,5 @@
     </collision>
   </link>
-  <link name="joint3">
+  <link name="link3">
     <visual>
       <geometry>
@@ -58,5 +58,5 @@
     </collision>
   </link>
-  <link name="joint4">
+  <link name="link4">
     <visual>
       <geometry>
@@ -72,5 +72,5 @@
     </collision>
   </link>
-  <link name="joint5">
+  <link name="link5">
     <visual>
       <geometry>
@@ -86,8 +86,8 @@
     </collision>
   </link>
-  <link name="endeffector">
+  <link name="gripper">
     <visual>
       <geometry>
-       <mesh filename="package://mycobot_description/urdf/myarm_c650/endeffector.dae"/>
+       <mesh filename="package://mycobot_description/urdf/myarm_c650/myarm_c_grip_Base.dae"/>
       </geometry>
     <origin xyz = "0 0 0.003 " rpy = " 3.14159 0 0"/>
@@ -95,72 +95,95 @@
     <collision>
       <geometry>
-       <mesh filename="package://mycobot_description/urdf/myarm_c650/endeffector.dae"/>
+       <mesh filename="package://mycobot_description/urdf/myarm_c650/myarm_c_grip_Base.dae"/>
       </geometry>
     <origin xyz = "0 0 0.003 " rpy = " 3.14159 0 0"/>
     </collision>
   </link>
-  <!-- <link name="endeffector">
+  <link name="gripper_left">
     <visual>
       <geometry>
-       <mesh filename="package://mycobot_description/urdf/myarm_c650/endeffector.dae"/>
+       <mesh filename="package://mycobot_description/urdf/myarm_c650/myarm_c_grip_R.dae"/>
       </geometry>
-    <origin xyz = "0.0 0 -0.009 " rpy = " 0 0 -1.5708"/>
+    <origin xyz = "0.010 0 0 " rpy = " 1.5708 3.14159 -1.5708"/>
     </visual>
     <collision>
       <geometry>
-       <mesh filename="package://mycobot_description/urdf/myarm_c650/endeffector.dae"/>
+       <mesh filename="package://mycobot_description/urdf/myarm_c650/myarm_c_grip_R.dae"/>
       </geometry>
-    <origin xyz = "0.0 0 -0.009 " rpy = " 0 0 -1.5708"/>
+    <origin xyz = "0.010 0 0 " rpy = " 1.5708 3.14159 -1.5708"/>
     </collision>
-  </link> -->
-  <joint name="joint1_to_base" type="revolute">
+  </link>
+  <link name="gripper_right">
+    <visual>
+      <geometry>
+       <mesh filename="package://mycobot_description/urdf/myarm_c650/myarm_c_grip_L.dae"/>
+      </geometry>
+    <origin xyz = "0.010 0 0 " rpy = " 1.5708 3.14159 -1.5708"/>
+    </visual>
+    <collision>
+      <geometry>
+       <mesh filename="package://mycobot_description/urdf/myarm_c650/myarm_c_grip_L.dae"/>
+      </geometry>
+    <origin xyz = "0.010 0 0 " rpy = " 1.5708 3.14159 -1.5708"/>
+    </collision>
+  </link>
+  <joint name="joint1" type="revolute">
     <axis xyz="0 0 1"/>
     <limit effort = "1000.0" lower = "-2.7925" upper = "2.7925" velocity = "0"/>
     <parent link="base"/>
-    <child link="joint1"/>
+    <child link="link1"/>
     <origin xyz= "0 0 0.070" rpy = "3.14159 0 0"/>
   </joint>
-  <joint name="joint2_to_joint1" type="revolute">
+  <joint name="joint2" type="revolute">
     <axis xyz="0 0 1"/>
     <limit effort = "1000.0" lower = "-1.3962" upper = "1.3962" velocity = "0"/>
-    <parent link="joint1"/>
-    <child link="joint2"/>
+    <parent link="link1"/>
+    <child link="link2"/>
     <!-- <origin xyz= "0 0  0" rpy = "1.5708 3.14159 0"/>   -->
     <origin xyz= "0 0 -0.080" rpy = "1.5708 0 0"/>
   </joint>
-  <joint name="joint3_to_joint2" type="revolute">
+  <joint name="joint3" type="revolute">
     <axis xyz=" 0 0 1"/>
     <limit effort = "1000.0" lower = "-2.8797" upper = "2.8797" velocity = "0"/>
-    <parent link="joint2"/>
-    <child link="joint3"/>
+    <parent link="link2"/>
+    <child link="link3"/>
     <origin xyz= "0.0565 -0.296 0   " rpy = "0 0 0"/>
   </joint>
-  <joint name="joint4_to_joint3" type="revolute">
+  <joint name="joint4" type="revolute">
     <axis xyz=" 0 0 1"/>
     <limit effort = "1000.0" lower = "-1.7453" upper = "1.3962" velocity = "0"/>
-    <parent link="joint3"/>
-    <child link="joint4"/>
+    <parent link="link3"/>
+    <child link="link4"/>
     <origin xyz= "0.081 0 0.004" rpy = "0 -1.5708 0"/>
   </joint>
-  <joint name="joint5_to_joint4" type="revolute">
+  <joint name="joint5" type="revolute">
     <axis xyz="0 0 1"/>
     <limit effort = "1000.0" lower = "-2.8797" upper = "2.8797" velocity = "0"/>
-    <parent link="joint4"/>
-    <child link="joint5"/>
+    <parent link="link4"/>
+    <child link="link5"/>
     <origin xyz= "0.0 0.0003 -0.2595" rpy = "-1.5708 3.14159 -1.5708"/>
   </joint>
-  <joint name="endeffector_to_joint5" type="revolute">
+  <joint name="joint6" type="revolute">
     <axis xyz="0 0 1"/>
     <limit effort = "1000.0" lower = "-1.9198" upper = "1.9198" velocity = "0"/>
-    <parent link="joint5"/>
-    <child link="endeffector"/>
+    <parent link="link5"/>
+    <child link="gripper"/>
     <origin xyz= "0 -0.045 0" rpy = "-1.5708 0 0"/>
   </joint>
-  <!-- <joint name="endeffector_to_endeffector" type="revolute">
+  <joint name="gripper" type="prismatic">
     <axis xyz="0 0 1"/>
-    <limit effort = "1000.0" lower = "-2.8797" upper = "2.8797" velocity = "0"/>
-    <parent link="endeffector"/>
-    <child link="endeffector"/>
-    <origin xyz= "0 -0.056 0" rpy = "1.5708 0 0"/>
-  </joint> -->
+    <limit effort = "1000.0" lower = "0" upper = "0.022" velocity = "0"/>
+    <parent link="gripper"/>
+    <child link="gripper_left"/>
+    <origin xyz= "-0.030 0 -0.066" rpy = "3.14 -1.57 1.57"/>
+  </joint>
+  <joint name="gripper_r" type="prismatic">
+    <axis xyz="0 0 -1"/>
+    <limit effort = "1000.0" lower = "0" upper = "0.022" velocity = "0"/>
+    <parent link="gripper"/>
+    <child link="gripper_right"/>
+    <origin xyz= "-0.030 0 -0.066" rpy = "3.14 -1.57 1.57"/>
+    <!-- 跟随左手指运动 -->
+    <mimic joint="gripper" multiplier="1.0" offset="0" />
+  </joint>
 </robot>

File: mycobot_description/urdf/myarm_m/myarm_m.urdf (robot description, URDF)
Before this commit: robot myarm_m, 7 links, 6 joints
Links:
- removed link endeffector
- removed link joint1
- removed link joint2
- removed link joint3
- removed link joint4
- removed link joint5
- added link gripper; collision mesh filename=package://mycobot_description/urdf/myarm_m/finger_holder.dae; visual mesh filename=package://mycobot_description/urdf/myarm_m/finger_holder.dae
- added link gripper_left; collision mesh filename=package://mycobot_description/urdf/myarm_m/finger_left.dae; visual mesh filename=package://mycobot_description/urdf/myarm_m/finger_left.dae
- added link gripper_right; collision mesh filename=package://mycobot_description/urdf/myarm_m/finger_right.dae; visual mesh filename=package://mycobot_description/urdf/myarm_m/finger_right.dae
- added link link1; collision mesh filename=package://mycobot_description/urdf/myarm_m/link1.dae; visual mesh filename=package://mycobot_description/urdf/myarm_m/link1.dae
- added link link2; collision mesh filename=package://mycobot_description/urdf/myarm_m/link2.dae; visual mesh filename=package://mycobot_description/urdf/myarm_m/link2.dae
- added link link3; collision mesh filename=package://mycobot_description/urdf/myarm_m/link3.dae; visual mesh filename=package://mycobot_description/urdf/myarm_m/link3.dae
- added link link4; collision mesh filename=package://mycobot_description/urdf/myarm_m/link4.dae; visual mesh filename=package://mycobot_description/urdf/myarm_m/link4.dae
- added link link5; collision mesh filename=package://mycobot_description/urdf/myarm_m/link5.dae; visual mesh filename=package://mycobot_description/urdf/myarm_m/link5.dae
- link base: geometry collision mesh filename=package://mycobot_description/urdf/myarm_m/myarm_m_base.dae; visual mesh filename=package://mycobot_description/urdf/myarm_m/myarm_m_base.dae
Joints:
- removed joint endeffector_to_joint5
- removed joint joint1_to_base
- removed joint joint2_to_joint1
- removed joint joint3_to_joint2
- removed joint joint4_to_joint3
- removed joint joint5_to_joint4
- added joint gripper: type prismatic, parent gripper, child gripper_left, origin xyz=0.008 0 -0.036 rpy=-1.57 0 -1.57, axis 0 0 1, limit lower=0 upper=0.0345 effort=1000.0 velocity=0
- added joint gripper_r: type prismatic, parent gripper, child gripper_right, origin xyz=-0.008 0 -0.036 rpy=-1.57 0 -1.57, axis 0 0 -1, limit lower=0 upper=0.06 effort=1000.0 velocity=0, mimic joint=gripper multiplier=1.0 offset=0
- added joint joint1: type revolute, parent base, child link1, origin xyz=0 0 0 rpy=0 3.14 0, axis 0 0 1, limit lower=-3.0368 upper=2.9147 effort=1000.0 velocity=0
- added joint joint2: type revolute, parent link1, child link2, origin xyz=0 0 -0.175 rpy=-1.57079 -1.57079 0, axis 0 0 1, limit lower=-1.6057 upper=1.6232 effort=1000.0 velocity=0
- added joint joint3: type revolute, parent link2, child link3, origin xyz=-0.303 -0.057 0    rpy=0 3.14159 -1.57079, axis  0 0 1, limit lower=-1.5882 upper=1.7977 effort=1000.0 velocity=0
- added joint joint4: type revolute, parent link3, child link4, origin xyz=-0.08 0 0 rpy=0 1.57079 0, axis  0 0 1, limit lower=-2.9671 upper=2.9671 effort=1000.0 velocity=0
- added joint joint5: type revolute, parent link4, child link5, origin xyz=0 0 -0.258 rpy=0 1.57079 0, axis 0 0 1, limit lower=-1.6755 upper=1.5533 effort=1000.0 velocity=0
- added joint joint6: type revolute, parent link5, child gripper, origin xyz=0.07 0 0 rpy=0 -1.57079 0, axis 0 0 1, limit lower=-2.9671 upper=2.9671 effort=1000.0 velocity=0

File: mycobot_description/urdf/myarm_m/myarm_m.urdf.xacro (robot description, xacro)
@@ -5,5 +5,5 @@
   <visual>
     <geometry>
-     <mesh filename="package://mycobot_description/urdf/myarm_m/base.dae"/>
+     <mesh filename="package://mycobot_description/urdf/myarm_m/myarm_m_base.dae"/>
     </geometry>
     <origin xyz = "0.0 0 0 " rpy = " 0 0 0"/>
@@ -11,13 +11,13 @@
   <collision>
     <geometry>
-     <mesh filename="package://mycobot_description/urdf/myarm_m/base.dae"/>
+     <mesh filename="package://mycobot_description/urdf/myarm_m/myarm_m_base.dae"/>
       </geometry>
       <origin xyz = "0.0 0 0 " rpy = " 0 0 0"/>
   </collision>
 </link>
-<link name="joint1">
+<link name="link1">
   <visual>
     <geometry>
-     <mesh filename="package://mycobot_description/urdf/myarm_m/joint1.dae"/>
+     <mesh filename="package://mycobot_description/urdf/myarm_m/link1.dae"/>
     </geometry>
     <origin xyz = "0.0 0 -0.1 " rpy = " 0 3.14 0"/>
@@ -25,13 +25,13 @@
   <collision>
    <geometry>
-     <mesh filename="package://mycobot_description/urdf/myarm_m/joint1.dae"/>
+     <mesh filename="package://mycobot_description/urdf/myarm_m/link1.dae"/>
     </geometry>
     <origin xyz = "0.0 0 -0.1 " rpy = "0 3.14 0"/>
   </collision>
 </link>
-<link name="joint2">
+<link name="link2">
   <visual>
     <geometry>
-     <mesh filename="package://mycobot_description/urdf/myarm_m/joint2.dae"/>
+     <mesh filename="package://mycobot_description/urdf/myarm_m/link2.dae"/>
     </geometry>
   <origin xyz = "0.0 0 0 " rpy = "0 3.14159 0"/>
@@ -39,13 +39,13 @@
   <collision>
     <geometry>
-     <mesh filename="package://mycobot_description/urdf/myarm_m/joint2.dae"/>
+     <mesh filename="package://mycobot_description/urdf/myarm_m/link2.dae"/>
     </geometry>
     <origin xyz = "0.0 0 0 " rpy = "0 3.14159 0"/>
   </collision>
 </link>
-<link name="joint3">
+<link name="link3">
   <visual>
     <geometry>
-     <mesh filename="package://mycobot_description/urdf/myarm_m/joint3.dae"/>
+     <mesh filename="package://mycobot_description/urdf/myarm_m/link3.dae"/>
     </geometry>
     <origin xyz = "0.0 0 0" rpy = "0 3.14159 0"/>
@@ -53,13 +53,13 @@
   <collision>
     <geometry>
-     <mesh filename="package://mycobot_description/urdf/myarm_m/joint3.dae"/>
+     <mesh filename="package://mycobot_description/urdf/myarm_m/link3.dae"/>
     </geometry>
     <origin xyz = "0.0 0 0.0" rpy = "0 3.14159 0"/>
   </collision>
 </link>
-<link name="joint4">
+<link name="link4">
   <visual>
     <geometry>
-     <mesh filename="package://mycobot_description/urdf/myarm_m/joint4.dae"/>
+     <mesh filename="package://mycobot_description/urdf/myarm_m/link4.dae"/>
     </geometry>
   <origin xyz = "0.0 0 0 " rpy = " 0 3.14159 -1.5708"/>
@@ -67,13 +67,13 @@
   <collision>
      <geometry>
-     <mesh filename="package://mycobot_description/urdf/myarm_m/joint4.dae"/>
+     <mesh filename="package://mycobot_description/urdf/myarm_m/link4.dae"/>
     </geometry>
     <origin xyz = "0.0 0 0 " rpy = " 0 3.14159  -1.5708"/>
   </collision>
 </link>
-<link name="joint5">
+<link name="link5">
   <visual>
     <geometry>
-     <mesh filename="package://mycobot_description/urdf/myarm_m/joint5.dae"/>
+     <mesh filename="package://mycobot_description/urdf/myarm_m/link5.dae"/>
     </geometry>
   <origin xyz = "0 0.00 0" rpy = " 0 0 0"/>
@@ -81,13 +81,13 @@
   <collision>
     <geometry>
-     <mesh filename="package://mycobot_description/urdf/myarm_m/joint5.dae"/>
+     <mesh filename="package://mycobot_description/urdf/myarm_m/link5.dae"/>
     </geometry>
   <origin xyz = "0 0.00 0 " rpy = " 0 0 0"/>
   </collision>
 </link>
-<link name="endeffector">
+<link name="gripper">
   <visual>
     <geometry>
-     <mesh filename="package://mycobot_description/urdf/myarm_m/endeffector.dae"/>
+     <mesh filename="package://mycobot_description/urdf/myarm_m/finger_holder.dae"/>
     </geometry>
   <origin xyz = "0 0.00 0" rpy = " 0 3.14159 -1.57079"/>
@@ -95,50 +95,94 @@
   <collision>
     <geometry>
-     <mesh filename="package://mycobot_description/urdf/myarm_m/endeffector.dae"/>
+     <mesh filename="package://mycobot_description/urdf/myarm_m/finger_holder.dae"/>
     </geometry>
   <origin xyz = "0 0.00 0" rpy = " 0 3.14159 -1.57079"/>
   </collision>
 </link>
-<joint name="joint1_to_base" type="revolute">
+<link name="gripper_left">
+  <visual>
+    <geometry>
+     <mesh filename="package://mycobot_description/urdf/myarm_m/finger_left.dae"/>
+    </geometry>
+  <origin xyz = "0 0.00 0" rpy = " 0 3.14159 -1.57079"/>
+  </visual>
+  <collision>
+    <geometry>
+     <mesh filename="package://mycobot_description/urdf/myarm_m/finger_left.dae"/>
+    </geometry>
+  <origin xyz = "0 0.00 0" rpy = " 0 0 0"/>
+  </collision>
+</link>
+<link name="gripper_right">
+  <visual>
+    <geometry>
+     <mesh filename="package://mycobot_description/urdf/myarm_m/finger_right.dae"/>
+    </geometry>
+  <origin xyz = "0 0.00 0" rpy = " 0 3.14159 -1.57079"/>
+  </visual>
+  <collision>
+    <geometry>
+     <mesh filename="package://mycobot_description/urdf/myarm_m/finger_right.dae"/>
+    </geometry>
+  <origin xyz = "0 0.00 0" rpy = " 0 3.14159 -1.57079"/>
+  </collision>
+</link>
+<joint name="joint1" type="revolute">
   <axis xyz="0 0 1"/>
   <limit effort = "1000.0" lower = "-3.0368" upper = "2.9147" velocity = "0"/>
   <parent link="base"/>
-  <child link="joint1"/>
+  <child link="link1"/>
   <origin xyz= "0 0 0" rpy = "0 3.14 0"/>
 </joint>
-<joint name="joint2_to_joint1" type="revolute">
+<joint name="joint2" type="revolute">
   <axis xyz="0 0 1"/>
   <limit effort = "1000.0" lower = "-1.6057" upper = "1.6232" velocity = "0"/>
-  <parent link="joint1"/>
-  <child link="joint2"/>
+  <parent link="link1"/>
+  <child link="link2"/>
   <origin xyz= "0 0 -0.175" rpy = "-1.57079 -1.57079 0"/>
 </joint>
- <joint name="joint3_to_joint2" type="revolute">
+ <joint name="joint3" type="revolute">
   <axis xyz=" 0 0 1"/>
   <limit effort = "1000.0" lower = "-1.5882" upper = "1.7977" velocity = "0"/>
-  <parent link="joint2"/>
-  <child link="joint3"/>
+  <parent link="link2"/>
+  <child link="link3"/>
   <origin xyz= "-0.303 -0.057 0   " rpy = "0 3.14159 -1.57079"/>
 </joint>
-<joint name="joint4_to_joint3" type="revolute">
+<joint name="joint4" type="revolute">
   <axis xyz=" 0 0 1"/>
   <limit effort = "1000.0" lower = "-2.9671" upper = "2.9671" velocity = "0"/>
-  <parent link="joint3"/>
-  <child link="joint4"/>
+  <parent link="link3"/>
+  <child link="link4"/>
   <origin xyz= "-0.08 0 0" rpy = "0 1.57079 0"/>
 </joint>
-<joint name="joint5_to_joint4" type="revolute">
+<joint name="joint5" type="revolute">
   <axis xyz="0 0 1"/>
   <limit effort = "1000.0" lower = "-1.6755" upper = "1.5533" velocity = "0"/>
-  <parent link="joint4"/>
-  <child link="joint5"/>
+  <parent link="link4"/>
+  <child link="link5"/>
   <origin xyz= "0 0 -0.258" rpy = "0 1.57079 0"/>
 </joint>
-<joint name="endeffector_to_joint5" type="revolute">
+<joint name="joint6" type="revolute">
   <axis xyz="0 0 1"/>
   <limit effort = "1000.0" lower = "-2.9671" upper = "2.9671" velocity = "0"/>
-  <parent link="joint5"/>
-  <child link="endeffector"/>
+  <parent link="link5"/>
+  <child link="gripper"/>
   <origin xyz= "0.07 0 0" rpy = "0 -1.57079 0"/>
 </joint>
+<joint name="gripper" type="prismatic">
+  <axis xyz="0 0 1"/>
+  <limit effort = "1000.0" lower = "0" upper = "0.0345" velocity = "0"/>
+  <parent link="gripper"/>
+  <child link="gripper_left"/>
+  <origin xyz= "0.008 0 -0.036" rpy = "-1.57 0 -1.57"/>
+</joint>
+<joint name="gripper_r" type="prismatic">
+  <axis xyz="0 0 -1"/>
+  <limit effort = "1000.0" lower = "0" upper = "0.06" velocity = "0"/>
+  <parent link="gripper"/>
+  <child link="gripper_right"/>
+  <origin xyz= "-0.008 0 -0.036" rpy = "-1.57 0 -1.57"/>
+  <!-- 跟随左手指运动 -->
+  <mimic joint="gripper" multiplier="1.0" offset="0" />
+</joint>
 </robot>

Commit message: add s570 model follow segment

File: mycobot_description/urdf/myarm_c650/myarm_c650.urdf (robot description, URDF)
Before this commit: robot firefighter, 9 links, 8 joints
Joints:
- joint joint1: axis 0 0 1 -> 0 0 -1
- joint joint4: axis  0 0 1 ->  0 0 -1
- joint joint6: axis 0 0 1 -> 0 0 -1

File: mycobot_description/urdf/myarm_m/myarm_m.urdf (robot description, URDF)
Before this commit: robot myarm_m, 9 links, 8 joints
Joints:
- joint joint1: axis 0 0 1 -> 0 0 -1
- joint joint2: axis 0 0 1 -> 0 0 -1
- joint joint3: axis  0 0 1 ->  0 0 -1; limit lower=-1.5882 upper=1.7977 effort=1000.0 velocity=0 -> lower=-1.5882 upper=1.2977 effort=1000.0 velocity=0
- joint joint4: axis  0 0 1 ->  0 0 -1
- joint joint6: axis 0 0 1 -> 0 0 -1
