Commit message: improve ros1 myarmc650 code

File: mycobot_description/urdf/myarm_c650/myarm_c650.urdf.xacro (robot description, xacro)
@@ -11,5 +11,5 @@
     <collision>
       <geometry>
-       <mesh filename="package://mycobot_description/urdf/myarm_c650/bamyarm_basic_basese.dae"/>
+       <mesh filename="package://mycobot_description/urdf/myarm_c650/myarm_basic_base.dae"/>
         </geometry>
         <origin xyz = "0.0 0 0 " rpy = " 0 0 0"/>

Commit message: add MC_320 Case

File: mycobot_description/urdf/myarm_c650/myarm_c650.urdf.xacro (robot description, xacro)
@@ -129,5 +129,5 @@
   </link>
   <joint name="joint1" type="revolute">
-    <axis xyz="0 0 1"/>
+    <axis xyz="0 0 -1"/>
     <limit effort = "1000.0" lower = "-2.7925" upper = "2.7925" velocity = "0"/>
     <parent link="base"/>
@@ -151,5 +151,5 @@
   </joint>
   <joint name="joint4" type="revolute">
-    <axis xyz=" 0 0 1"/>
+    <axis xyz=" 0 0 -1"/>
     <limit effort = "1000.0" lower = "-1.7453" upper = "1.3962" velocity = "0"/>
     <parent link="link3"/>
@@ -165,5 +165,5 @@
   </joint>
   <joint name="joint6" type="revolute">
-    <axis xyz="0 0 1"/>
+    <axis xyz="0 0 -1"/>
     <limit effort = "1000.0" lower = "-1.9198" upper = "1.9198" velocity = "0"/>
     <parent link="link5"/>
