Commit message: 增加三指 320/630 moveit RVIZ跟随demo

File: mycobot_description/urdf/three_gripper/mycobot_pro_three_gripper.urdf (robot description, URDF)
Before this commit: robot firefighter, 1 links, 0 joints
Links:
- link gripper_base: geometry collision mesh filename=package://mycobot_description/urdf/three_gripper/three_myha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; visual mesh filename=package://mycobot_description/urdf/three_gripper/three_myha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
