Commit message: 320 力控夹爪增加连接件模型

File: mycobot_320/new_mycobot_320_force_gripper_moveit/config/gazebo_firefighter.urdf (robot description, URDF)
Before this commit: robot firefighter, 14 links, 13 joints
Links:
- added link gripper_connection, mass 0.1; collision mesh filename=package://mycobot_description/urdf/mycobot_320_m5_2022/forc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; visual mesh filename=package://mycobot_description/urdf/mycobot_320_m5_2022/forc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
Joints:
- added joint joint6output_to_gripper_connect: type fixed, parent link6, child gripper_connection, origin xyz=0 0.0 0.011 rpy=0 0 0
- joint joint6output_to_gripper_base: origin xyz=0 0.0 0.034 rpy=1.5708 0 0 -> xyz=0 -0.02 0.036 rpy=1.5708 0 0; parent link6 -> gripper_connection

File: mycobot_description/urdf/mycobot_320_m5_2022/pro_320_m5_2022_force_gripper.urdf (robot description, URDF)
Before this commit: robot firefighter, 14 links, 13 joints
Links:
- added link gripper_connection; collision mesh filename=package://mycobot_description/urdf/mycobot_320_m5_2022/forc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; visual mesh filename=package://mycobot_description/urdf/mycobot_320_m5_2022/forc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
Joints:
- added joint joint6output_to_gripper_connect: type fixed, parent link6, child gripper_connection, origin xyz=0 0.0 0.01 rpy=0 0 0
- joint joint6output_to_gripper_base: origin xyz=0 0.0 0.034 rpy=1.5708 0 0 -> xyz=0 -0.02 0.036 rpy=1.5708 0 0; parent link6 -> gripper_connection

File: mycobot_description/urdf/mycobot_320_m5_2022/pro_320_m5_2022_moveit_force_gripper.urdf (robot description, URDF)
Before this commit: robot firefighter, 14 links, 13 joints
Links:
- added link gripper_connection; collision mesh filename=package://mycobot_description/urdf/mycobot_320_m5_2022/forc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; visual mesh filename=package://mycobot_description/urdf/mycobot_320_m5_2022/forc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
Joints:
- added joint joint6output_to_gripper_connect: type fixed, parent link6, child gripper_connection, origin xyz=0 0.0 0.011 rpy=0 0 0
- joint joint6output_to_gripper_base: origin xyz=0 0.0 0.034 rpy=1.5708 0 0 -> xyz=0 -0.02 0.036 rpy=1.5708 0 0; parent link6 -> gripper_connection

File: mycobot_description/urdf/mycobot_320_pi_2022/pro_320_pi_2022_force_gripper.urdf (robot description, URDF)
Before this commit: robot firefighter, 14 links, 13 joints
Links:
- added link gripper_connection; collision mesh filename=package://mycobot_description/urdf/mycobot_320_pi_2022/forc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; visual mesh filename=package://mycobot_description/urdf/mycobot_320_pi_2022/forc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
Joints:
- added joint joint6output_to_gripper_connect: type fixed, parent link6, child gripper_connection, origin xyz=0 0.0 0.0 rpy=0 0 0
- joint joint6output_to_gripper_base: origin xyz=0 0.0 0.026 rpy=1.5708 0 0 -> xyz=0 -0.02 0.036 rpy=1.5708 0 0; parent link6 -> gripper_connection

File: mycobot_description/urdf/mycobot_320_pi_2022/pro_320_pi_2022_moveit_force_gripper.urdf (robot description, URDF)
Before this commit: robot firefighter, 14 links, 13 joints
Links:
- added link gripper_connection; collision mesh filename=package://mycobot_description/urdf/mycobot_320_pi_2022/forc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; visual mesh filename=package://mycobot_description/urdf/mycobot_320_pi_2022/forc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
Joints:
- added joint joint6output_to_gripper_connect: type fixed, parent link6, child gripper_connection, origin xyz=0 0.0 0.0 rpy=0 0 0
- joint joint6output_to_gripper_base: origin xyz=0 0.0 0.026 rpy=1.5708 0 0 -> xyz=0 -0.02 0.036 rpy=1.5708 0 0; parent link6 -> gripper_connection
