Commit message: 修复280PI urdf j4、j5

File: mycobot_description/urdf/mycobot_280_pi/mycobot_280_pi.urdf (robot description, URDF)
Before this commit: robot firefighter, 8 links, 7 joints
Joints:
- joint joint6_to_joint5: origin xyz=0 -0.07318 0 rpy=1.5708 -1.5708 0 -> xyz=0 -0.07318 -0.001 rpy=1.5708 -1.5708 0

File: mycobot_description/urdf/mycobot_280_pi/mycobot_280pi_with_camera_flange.urdf (robot description, URDF)
Before this commit: robot firefighter, 9 links, 8 joints
Joints:
- joint joint6_to_joint5: origin xyz=0 -0.07318 0 rpy=1.5708 -1.5708 0 -> xyz=0 -0.07318 -0.001 rpy=1.5708 -1.5708 0

File: mycobot_description/urdf/mycobot_280_pi/mycobot_280pi_with_camera_flange_pump.urdf (robot description, URDF)
Before this commit: robot firefighter, 11 links, 10 joints
Joints:
- joint joint6_to_joint5: origin xyz=0 -0.07318 0 rpy=1.5708 -1.5708 0 -> xyz=0 -0.07318 -0.001 rpy=1.5708 -1.5708 0

File: mycobot_description/urdf/mycobot_280_pi/mycobot_280pi_with_pump.urdf (robot description, URDF)
Before this commit: robot firefighter, 10 links, 9 joints
Joints:
- joint joint6_to_joint5: origin xyz=0 -0.07318 0 rpy=1.5708 -1.5708 0 -> xyz=0 -0.07318 -0.001 rpy=1.5708 -1.5708 0

File: mycobot_description/urdf/mycobot_280_pi/mycobot_280pi_with_vision_v2.urdf (robot description, URDF)
Before this commit: robot mycobot_ai, 8 links, 7 joints
Joints:
- joint joint6_to_joint5: origin xyz=0 -0.07318 0 rpy=1.5708 -1.5708 0 -> xyz=0 -0.07318 -0.001 rpy=1.5708 -1.5708 0
