Commit message: 更新280系列urdf关节限位

File: mycobot_description/urdf/mycobot_280_m5/mycobot_280m5_with_gripper_parallel.urdf (robot description, URDF)
Before this commit: robot firefighter, 15 links, 14 joints
Joints:
- joint joint2_to_joint1: limit lower=-2.879793 upper=2.879793 effort=1000.0 velocity=0 -> lower=-2.9321 upper=2.9321 effort=1000.0 velocity=0
- joint joint3_to_joint2: limit lower=-2.879793 upper=2.879793 effort=1000.0 velocity=0 -> lower=-2.3561 upper=2.3561 effort=1000.0 velocity=0
- joint joint4_to_joint3: limit lower=-2.879793 upper=2.879793 effort=1000.0 velocity=0 -> lower=-2.6179 upper=2.6179 effort=1000.0 velocity=0
- joint joint5_to_joint4: limit lower=-2.879793 upper=2.879793 effort=1000.0 velocity=0 -> lower=-2.5307 upper=2.5307 effort=1000.0 velocity=0
- joint joint6output_to_joint6: limit lower=-3.05 upper=3.05 effort=1000.0 velocity=0 -> lower=-3.14 upper=3.14 effort=1000.0 velocity=0

File: mycobot_description/urdf/mycobot_280_pi/mycobot_280_pi.urdf (robot description, URDF)
Before this commit: robot firefighter, 8 links, 7 joints
Joints:
- joint joint2_to_joint1: limit lower=-3.14 upper=3.14159 effort=1000.0 velocity=0 -> lower=-2.9321 upper=2.9321 effort=1000.0 velocity=0
- joint joint3_to_joint2: limit lower=-3.14 upper=3.14159 effort=1000.0 velocity=0 -> lower=-2.3561 upper=2.3561 effort=1000.0 velocity=0
- joint joint4_to_joint3: limit lower=-3.14 upper=3.14159 effort=1000.0 velocity=0 -> lower=-2.6179 upper=2.6179 effort=1000.0 velocity=0
- joint joint5_to_joint4: limit lower=-3.14 upper=3.14159 effort=1000.0 velocity=0 -> lower=-2.5307 upper=2.5307 effort=1000.0 velocity=0
- joint joint6_to_joint5: limit lower=-3.14 upper=3.14159 effort=1000.0 velocity=0 -> lower=-2.8797 upper=2.8797 effort=1000.0 velocity=0

File: mycobot_description/urdf/mycobot_280_pi/mycobot_280pi_with_camera_flange.urdf (robot description, URDF)
Before this commit: robot firefighter, 9 links, 8 joints
Joints:
- joint joint2_to_joint1: limit lower=-3.14 upper=3.14159 effort=1000.0 velocity=0 -> lower=-2.9321 upper=2.9321 effort=1000.0 velocity=0
- joint joint3_to_joint2: limit lower=-3.14 upper=3.14159 effort=1000.0 velocity=0 -> lower=-2.3561 upper=2.3561 effort=1000.0 velocity=0
- joint joint4_to_joint3: limit lower=-3.14 upper=3.14159 effort=1000.0 velocity=0 -> lower=-2.6179 upper=2.6179 effort=1000.0 velocity=0
- joint joint5_to_joint4: limit lower=-3.14 upper=3.14159 effort=1000.0 velocity=0 -> lower=-2.5307 upper=2.5307 effort=1000.0 velocity=0
- joint joint6_to_joint5: limit lower=-3.14 upper=3.14159 effort=1000.0 velocity=0 -> lower=-2.8797 upper=2.8797 effort=1000.0 velocity=0

File: mycobot_description/urdf/mycobot_280_pi/mycobot_280pi_with_camera_flange_pump.urdf (robot description, URDF)
Before this commit: robot firefighter, 11 links, 10 joints
Joints:
- joint joint2_to_joint1: limit lower=-3.14 upper=3.14159 effort=1000.0 velocity=0 -> lower=-2.9321 upper=2.9321 effort=1000.0 velocity=0
- joint joint3_to_joint2: limit lower=-3.14 upper=3.14159 effort=1000.0 velocity=0 -> lower=-2.3561 upper=2.3561 effort=1000.0 velocity=0
- joint joint4_to_joint3: limit lower=-3.14 upper=3.14159 effort=1000.0 velocity=0 -> lower=-2.6179 upper=2.6179 effort=1000.0 velocity=0
- joint joint5_to_joint4: limit lower=-3.14 upper=3.14159 effort=1000.0 velocity=0 -> lower=-2.5307 upper=2.5307 effort=1000.0 velocity=0
- joint joint6_to_joint5: limit lower=-3.14 upper=3.14159 effort=1000.0 velocity=0 -> lower=-2.8797 upper=2.8797 effort=1000.0 velocity=0

File: mycobot_description/urdf/mycobot_280_pi/mycobot_280pi_with_pump.urdf (robot description, URDF)
Before this commit: robot firefighter, 10 links, 9 joints
Joints:
- joint joint2_to_joint1: limit lower=-3.14 upper=3.14159 effort=1000.0 velocity=0 -> lower=-2.9321 upper=2.9321 effort=1000.0 velocity=0
- joint joint3_to_joint2: limit lower=-3.14 upper=3.14159 effort=1000.0 velocity=0 -> lower=-2.3561 upper=2.3561 effort=1000.0 velocity=0
- joint joint4_to_joint3: limit lower=-3.14 upper=3.14159 effort=1000.0 velocity=0 -> lower=-2.6179 upper=2.6179 effort=1000.0 velocity=0
- joint joint5_to_joint4: limit lower=-3.14 upper=3.14159 effort=1000.0 velocity=0 -> lower=-2.5307 upper=2.5307 effort=1000.0 velocity=0
- joint joint6_to_joint5: limit lower=-3.14 upper=3.14159 effort=1000.0 velocity=0 -> lower=-2.8797 upper=2.8797 effort=1000.0 velocity=0

File: mycobot_description/urdf/mycobot_280_pi/mycobot_280pi_with_vision_v2.urdf (robot description, URDF)
Before this commit: robot mycobot_ai, 8 links, 7 joints
Joints:
- joint joint2_to_joint1: limit lower=-3.14 upper=3.14159 effort=1000.0 velocity=0 -> lower=-2.9321 upper=2.9321 effort=1000.0 velocity=0
- joint joint3_to_joint2: limit lower=-3.14 upper=3.14159 effort=1000.0 velocity=0 -> lower=-2.3561 upper=2.3561 effort=1000.0 velocity=0
- joint joint4_to_joint3: limit lower=-3.14 upper=3.14159 effort=1000.0 velocity=0 -> lower=-2.6179 upper=2.6179 effort=1000.0 velocity=0
- joint joint5_to_joint4: limit lower=-3.14 upper=3.14159 effort=1000.0 velocity=0 -> lower=-2.5307 upper=2.5307 effort=1000.0 velocity=0
- joint joint6_to_joint5: limit lower=-3.14 upper=3.14159 effort=1000.0 velocity=0 -> lower=-2.8797 upper=2.8797 effort=1000.0 velocity=0

Commit message: Fixed the 280M5 gripper moveit collision gripper problem (parallel installation)

File: mycobot_description/urdf/mycobot_280_m5/mycobot_280m5_with_gripper_parallel.urdf (robot description, URDF)
Before this commit: robot firefighter, 15 links, 14 joints
Links:
- link g_base: mass None -> 0.1
- link gripper_base: mass None -> 0.1; geometry collision cylinder length=0.01 radius=0.02; visual mesh filename=package://mycobot_description/urdf/mycobot_280_m5/gripper_b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
- link gripper_left1: mass None -> 0.1; geometry collision cylinder length=0.005 radius=0.0034; visual mesh filename=package://mycobot_description/urdf/mycobot_280_m5/gripper_l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
- link gripper_left2: mass None -> 0.1; geometry collision cylinder length=0.005 radius=0.0034; visual mesh filename=package://mycobot_description/urdf/mycobot_280_m5/gripper_l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
- link gripper_left3: mass None -> 0.1; geometry collision cylinder length=0.003 radius=0.0034; visual mesh filename=package://mycobot_description/urdf/mycobot_280_m5/gripper_l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
- link gripper_right1: mass None -> 0.1; geometry collision cylinder length=0.005 radius=0.0034; visual mesh filename=package://mycobot_description/urdf/mycobot_280_m5/gripper_r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
- link gripper_right2: mass None -> 0.1; geometry collision cylinder length=0.005 radius=0.0034; visual mesh filename=package://mycobot_description/urdf/mycobot_280_m5/gripper_r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
- link gripper_right3: mass None -> 0.1; geometry collision cylinder length=0.003 radius=0.0034; visual mesh filename=package://mycobot_description/urdf/mycobot_280_m5/gripper_r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
- link joint1: mass None -> 0.1
- link joint2: mass None -> 0.1
- link joint3: mass None -> 0.1
- link joint4: mass None -> 0.1
- link joint5: mass None -> 0.1
- link joint6: mass None -> 0.1
- link joint6_flange: mass None -> 0.1
Joints:
- joint gripper_controller: limit lower=-0.7 upper=0.15 effort=1000.0 velocity=0 -> lower=-0.78 upper=0.15 effort=1000.0 velocity=0
