Commit message: Add max velocity to mycobot 280 m5 model

File: mycobot_description/urdf/mycobot_280_m5/mycobot_280_m5.urdf (robot description, URDF)
Before this commit: robot firefighter, 8 links, 7 joints
Joints:
- joint joint2_to_joint1: limit lower=-2.9321 upper=2.9321 effort=1000.0 velocity=0 -> lower=-2.9321 upper=2.9321 effort=1000.0 velocity=2.792526803190927
- joint joint3_to_joint2: limit lower=-2.4434 upper=2.4434 effort=1000.0 velocity=0 -> lower=-2.4434 upper=2.4434 effort=1000.0 velocity=2.792526803190927
- joint joint4_to_joint3: limit lower=-2.6179 upper=2.6179 effort=1000.0 velocity=0 -> lower=-2.6179 upper=2.6179 effort=1000.0 velocity=2.792526803190927
- joint joint5_to_joint4: limit lower=-2.6179 upper=2.6179 effort=1000.0 velocity=0 -> lower=-2.6179 upper=2.6179 effort=1000.0 velocity=2.792526803190927
- joint joint6_to_joint5: limit lower=-2.7052 upper=2.7925 effort=1000.0 velocity=0 -> lower=-2.7052 upper=2.7925 effort=1000.0 velocity=2.792526803190927
- joint joint6output_to_joint6: limit lower=-3.14 upper=3.14159 effort=1000.0 velocity=0 -> lower=-3.14 upper=3.14159 effort=1000.0 velocity=2.792526803190927
