Commit message: 新增 mycobot600 机械臂跟随仿真运动

File: mycobot_description/urdf/mycobot_pro_600/mycobot_pro_600_gripper.urdf (robot description, URDF)
Before this commit: robot firefighter, 16 links, 15 joints
Joints:
- joint joint3_to_joint2: origin xyz=0 0.04  0.085 rpy=1.5708 0 0 -> xyz=0 0.04  0.085 rpy=1.5706 1.5706 0
- joint joint5_to_joint4: origin xyz=0 0.25  0.025 rpy=0 0 0 -> xyz=0 0.25  0.025 rpy=0 0 -1.5706
- joint joint6output_to_tool1: type revolute -> fixed

File: mycobot_description/urdf/mycobot_pro_630/mycobot_630_gripper.urdf (robot description, URDF)
Before this commit: robot firefighter, 16 links, 15 joints
Joints:
- joint joint1_to_base: axis 0 0 -1 -> 0 0 1
- joint joint2_to_joint1: axis 0 0 -1 -> 0 0 1; origin xyz=0 0.06  0.038 rpy=1.5707 0 3.14159 -> xyz=0 0.06  0.038 rpy=1.5707 -1.5706 3.14159
- joint joint3_to_joint2: axis  0 0 -1 ->  0 0 1
- joint joint4_to_joint3: axis  0 0 -1 ->  0 0 1; origin xyz=0 0.2663 0    rpy=0 0 0 -> xyz=0 0.2663 0    rpy=0 0 1.5706
- joint joint5_to_joint4: origin xyz=0 0.055 0.039 rpy=1.5707 -1.5707 0 -> xyz=0 0.055 0.039 rpy=1.5707 0 0
- joint joint6output_to_tool1: type revolute -> fixed

Commit message: 优化600带夹爪实现moveit

File: mycobot_description/urdf/mycobot_pro_600/mycobot_pro_600_gripper.urdf (robot description, URDF)
Before this commit: robot firefighter, 16 links, 15 joints
Links:
- removed link tool1
- link base: geometry collision mesh filename=package://mycobot_description/urdf/mycobot_pro_600/J1-W.dae; visual mesh filename=package://mycobot_description/urdf/mycobot_pro_600/J1-W.dae
- link link1: geometry collision mesh filename=package://mycobot_description/urdf/mycobot_pro_600/J2-W.dae; visual mesh filename=package://mycobot_description/urdf/mycobot_pro_600/J2-W.dae
- link link2: geometry collision mesh filename=package://mycobot_description/urdf/mycobot_pro_600/J3-W.dae; visual mesh filename=package://mycobot_description/urdf/mycobot_pro_600/J3-W.dae
- link link3: geometry collision mesh filename=package://mycobot_description/urdf/mycobot_pro_600/J4-W.dae; visual mesh filename=package://mycobot_description/urdf/mycobot_pro_600/J4-W.dae
- link link4: geometry collision mesh filename=package://mycobot_description/urdf/mycobot_pro_600/J5-W.dae; visual mesh filename=package://mycobot_description/urdf/mycobot_pro_600/J5-W.dae
- link link5: geometry collision mesh filename=package://mycobot_description/urdf/mycobot_pro_600/J6-W.dae; visual mesh filename=package://mycobot_description/urdf/mycobot_pro_600/J6-W.dae
- link link6: geometry collision mesh filename=package://mycobot_description/urdf/mycobot_pro_600/J7-W.dae; visual mesh filename=package://mycobot_description/urdf/mycobot_pro_600/J7-W.dae
Joints:
- removed joint joint6output_to_tool1
- removed joint tool1_to_tool2
- added joint joint6output_to_tool2: type fixed, parent link6, child tool2, origin xyz=-0.016 0.0 0.0 rpy=-1.5706 0 1.5706, axis 0 1 0, limit lower=-3.05 upper=3.05 effort=1000.0 velocity=0
- joint joint3_to_joint2: origin xyz=0 0.04  0.085 rpy=1.5706 1.5706 0 -> xyz=0 0.042  0.072 rpy=1.5708 1.5706 0
- joint joint4_to_joint3: origin xyz=0.0 0.25 0    rpy=0 0 0 -> xyz=0.0 0.25 0.005    rpy=0 0 0
- joint joint6_to_joint5: origin xyz=0 0.058 -0.05 rpy=1.57080 -1.57080 3.14159 -> xyz=0 0.058 -0.052 rpy=1.57080 -1.57080 3.14159
- joint joint6output_to_joint6: origin xyz=-0.076 0 0.05 rpy=-1.57080 0 0  -> xyz=-0.06 0 0.048 rpy=-1.57080 0 0 
- joint tool2_to_gripper_base: origin xyz=0.0 0.0 0.04 rpy=1.5706 0 1.5706 -> xyz=0.005 0.0 0.047 rpy=1.5706 0 1.5706

Commit message: Fixed the problem of pro600_gripper_moveit joints accidentally colliding

File: mycobot_description/urdf/mycobot_pro_600/mycobot_pro_600_gripper.urdf (robot description, URDF)
Before this commit: robot firefighter, 15 links, 14 joints
Links:
- link base: geometry collision cylinder length=0.06 radius=0.038; visual mesh filename=package://mycobot_description/urdf/mycobot_pro_600/J1-W.dae
- link gripper_base: geometry collision cylinder length=0.03 radius=0.026; visual mesh filename=package://mycobot_description/urdf/mycobot_320_m5_2022/grip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
- link gripper_left1: geometry collision cylinder length=0.005 radius=0.004; visual mesh filename=package://mycobot_description/urdf/mycobot_320_m5_2022/grip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
- link gripper_left2: geometry collision cylinder length=0.003 radius=0.003; visual mesh filename=package://mycobot_description/urdf/mycobot_320_m5_2022/grip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
- link gripper_left3: geometry collision cylinder length=0.003 radius=0.018; visual mesh filename=package://mycobot_description/urdf/mycobot_320_m5_2022/grip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
- link gripper_right1: geometry collision cylinder length=0.005 radius=0.004; visual mesh filename=package://mycobot_description/urdf/mycobot_320_m5_2022/grip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
- link gripper_right2: geometry collision cylinder length=0.003 radius=0.003; visual mesh filename=package://mycobot_description/urdf/mycobot_320_m5_2022/grip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
- link gripper_right3: geometry collision cylinder length=0.003 radius=0.018; visual mesh filename=package://mycobot_description/urdf/mycobot_320_m5_2022/grip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
- link link1: geometry collision cylinder length=0.05 radius=0.03; visual mesh filename=package://mycobot_description/urdf/mycobot_pro_600/J2-W.dae
- link link2: geometry collision cylinder length=0.28 radius=0.024; visual mesh filename=package://mycobot_description/urdf/mycobot_pro_600/J3-W.dae
- link link3: geometry collision cylinder length=0.24 radius=0.024; visual mesh filename=package://mycobot_description/urdf/mycobot_pro_600/J4-W.dae
- link link4: geometry collision cylinder length=0.05 radius=0.024; visual mesh filename=package://mycobot_description/urdf/mycobot_pro_600/J5-W.dae
- link link5: geometry collision cylinder length=0.05 radius=0.028; visual mesh filename=package://mycobot_description/urdf/mycobot_pro_600/J6-W.dae
- link link6: geometry collision cylinder length=0.006 radius=0.026; visual mesh filename=package://mycobot_description/urdf/mycobot_pro_600/J7-W.dae
- link tool2: geometry collision cylinder length=0.006 radius=0.026; visual mesh filename=package://mycobot_description/urdf/mycobot_pro_600/tool2-mm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
