Commit message: fix 320 pi moveit urdf

File: mycobot_description/urdf/mycobot_320_pi_2022/new_mycobot_pro_320_pi_moveit_2022.urdf (robot description, URDF)
Before this commit: robot firefighter, 7 links, 6 joints
Joints:
- joint joint5_to_joint4: origin xyz=0.120  0.08878 rpy=0 0 1.57080 -> xyz=0.120 0 0.08878 rpy=0 0 1.57080
