Commit message: perf(p1-urdf):P1 optimizes the URDF file to achieve joint linkage control.

File: mycobot_description/urdf/ultraArm_p1/ultraArm_p1.urdf (robot description, URDF)
Before this commit: robot firefighter, 5 links, 4 joints
Links:
- removed link base
- removed link link1
- removed link link2
- removed link link3
- removed link link4
- added link FIX1, mass 0.000785398163397449; collision mesh filename=package://mycobot_description/urdf/ultraArm_p1/meshes/FIX1.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; visual mesh filename=package://mycobot_description/urdf/ultraArm_p1/meshes/FIX1.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
- added link FIX2, mass 0.000785398163397448; collision mesh filename=package://mycobot_description/urdf/ultraArm_p1/meshes/FIX2.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; visual mesh filename=package://mycobot_description/urdf/ultraArm_p1/meshes/FIX2.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
- added link FIX3, mass 0.000785398163397449; collision mesh filename=package://mycobot_description/urdf/ultraArm_p1/meshes/FIX3.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; visual mesh filename=package://mycobot_description/urdf/ultraArm_p1/meshes/FIX3.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
- added link J1-LINK, mass 0.36023578514819; collision mesh filename=package://mycobot_description/urdf/ultraArm_p1/meshes/J1-LI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; visual mesh filename=package://mycobot_description/urdf/ultraArm_p1/meshes/J1-LI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
- added link J2-Link3, mass 0.000785398163397449; collision mesh filename=package://mycobot_description/urdf/ultraArm_p1/meshes/J2-Li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; visual mesh filename=package://mycobot_description/urdf/ultraArm_p1/meshes/J2-Li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
- added link J2_Link1, mass 0.0305283235625227; collision mesh filename=package://mycobot_description/urdf/ultraArm_p1/meshes/J2_Li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; visual mesh filename=package://mycobot_description/urdf/ultraArm_p1/meshes/J2_Li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
- added link J2_Link2, mass 0.0757843800054117; collision mesh filename=package://mycobot_description/urdf/ultraArm_p1/meshes/J2_Li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; visual mesh filename=package://mycobot_description/urdf/ultraArm_p1/meshes/J2_Li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
- added link J2_Link4, mass 0.0263910621420943; collision mesh filename=package://mycobot_description/urdf/ultraArm_p1/meshes/J2_Li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; visual mesh filename=package://mycobot_description/urdf/ultraArm_p1/meshes/J2_Li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
- added link J3-LIink2, mass 0.0559892080648003; collision mesh filename=package://mycobot_description/urdf/ultraArm_p1/meshes/J3-LI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; visual mesh filename=package://mycobot_description/urdf/ultraArm_p1/meshes/J3-LI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
- added link J3_Link1, mass 0.0260308258274982; collision mesh filename=package://mycobot_description/urdf/ultraArm_p1/meshes/J3_Li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; visual mesh filename=package://mycobot_description/urdf/ultraArm_p1/meshes/J3_Li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
- added link J3_Link3, mass 0.0686504291131459; collision mesh filename=package://mycobot_description/urdf/ultraArm_p1/meshes/J3_Li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; visual mesh filename=package://mycobot_description/urdf/ultraArm_p1/meshes/J3_Li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
- added link J3_Link4, mass 0.000785398163397448; collision mesh filename=package://mycobot_description/urdf/ultraArm_p1/meshes/J3_Li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; visual mesh filename=package://mycobot_description/urdf/ultraArm_p1/meshes/J3_Li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
- added link J4_Link, mass 0.00784859322698103; collision mesh filename=package://mycobot_description/urdf/ultraArm_p1/meshes/J4_Li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; visual mesh filename=package://mycobot_description/urdf/ultraArm_p1/meshes/J4_Li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
- added link base_link, mass 0.627583870747359; collision mesh filename=package://mycobot_description/urdf/ultraArm_p1/meshes/base_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; visual mesh filename=package://mycobot_description/urdf/ultraArm_p1/meshes/base_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
- added link world
Joints:
- removed joint joint1
- removed joint joint2
- removed joint joint3
- removed joint joint4
- added joint F1: type fixed, parent J2_Link4, child FIX1, origin xyz=0.14231924206961 -0.00990000000000155 -0.00499078358865856 rpy=0 0 0, axis 0 0 0
- added joint F2: type fixed, parent J3_Link3, child FIX2, origin xyz=0.0250007533101423 0 0.024999246667158 rpy=0 0 0, axis 0 0 0
- added joint F3: type fixed, parent J2_Link4, child FIX3, origin xyz=0.0274097939152648 -0.0149000000000027 0.0250219973774115 rpy=0 0 0, axis 0 0 0
- added joint J1: type revolute, parent base_link, child J1-LINK, origin xyz=0 0 0.0860000000000012 rpy=0 0 0, axis 0 0 1, limit lower=-2.97 upper=2.97 effort=100 velocity=1
- added joint J2: type revolute, parent J1-LINK, child J2_Link1, origin xyz=0.0225 -0.015 0.0799 rpy=0 0 0, axis 0 1 0, limit lower=-0.35 upper=1.3962 effort=100 velocity=1
- added joint J2-2: type revolute, parent J1-LINK, child J2_Link2, origin xyz=-0.0025 -0.024 0.1049 rpy=0 0 0, axis 0 1 0, limit lower=-0.35 upper=1.3962 effort=100 velocity=1, mimic joint=J2 multiplier=1 offset=0
- added joint J2-3: type revolute, parent J2_Link2, child J2-Link3, origin xyz=0 0 0.14 rpy=0 0 0, axis 0 1 0, limit lower=1.3962 upper=0.35 effort=100 velocity=1, mimic joint=J2 multiplier=-1 offset=0
- added joint J2-4: type revolute, parent J2_Link1, child J2_Link4, origin xyz=-0.002409 0.0059 0.13998 rpy=0 0 0, axis 0 1 0, limit lower=-1.3962 upper=0.35 effort=100 velocity=1, mimic joint=J2-3 multiplier=1 offset=0
- added joint J3: type revolute, parent J2_Link4, child J3_Link1, origin xyz=0 0 0 rpy=0 0 0, axis 0 1 0, limit lower=0 upper=1.92 effort=100 velocity=1
- added joint J3-2: type revolute, parent FIX3, child J3-LIink2, origin xyz=0 0 0 rpy=0 0 0, axis 0 1 0, limit lower=0 upper=1.92 effort=100 velocity=1, mimic joint=J3 multiplier=1 offset=0
- added joint J3-3: type revolute, parent J3_Link1, child J3_Link3, origin xyz=0.14232 -0.0099 -0.0049908 rpy=0 0 0, axis 0 1 0, limit lower=-1.92 upper=0 effort=100 velocity=1, mimic joint=J3 multiplier=-1 offset=0
- added joint J3-4: type revolute, parent J3-LIink2, child J3_Link4, origin xyz=0.13991 0.005 -0.0050135 rpy=0 0 0, axis 0 1 0, limit lower=-1.92 upper=0 effort=100 velocity=1, mimic joint=J3-3 multiplier=1 offset=0
- added joint J4: type revolute, parent J3_Link3, child J4_Link, origin xyz=0.067813 0.019 -0.047739 rpy=0 0 0, axis 3.005E-05 0 1, limit lower=-3.14 upper=3.14 effort=100 velocity=1
- added joint world_to_base: type fixed, parent world, child base_link, origin xyz=0 0 0 rpy=0 0 0

File: mycobot_description/urdf/ultraArm_p1/ultraArm_p1_new.urdf (robot description, URDF)
Before this commit: robot firefighter, 11 links, 10 joints
Joints:
- joint joint3: limit lower=0 upper=0.5235 effort=1000.0 velocity=0 -> lower=0 upper=1.9198 effort=1000.0 velocity=0
- joint joint4: limit lower=-6.2831 upper=6.2831 effort=1000.0 velocity=0 -> lower=-3.14 upper=3.14 effort=1000.0 velocity=0

Commit message: fix(p1-urdf): update urdf file

File: mycobot_description/urdf/ultraArm_p1/ultraArm_p1.urdf (robot description, URDF)
Before this commit: robot firefighter, 15 links, 14 joints
Links:
- removed link J1-LINK
- removed link J2-Link3
- removed link J3-LIink2
- added link J1_LINK, mass 0.36023578514819; collision mesh filename=package://mycobot_description/urdf/ultraArm_p1/J1_LINK.STL; visual mesh filename=package://mycobot_description/urdf/ultraArm_p1/J1_LINK.STL
- added link J2_Link3, mass 0.000785398163397449; collision mesh filename=package://mycobot_description/urdf/ultraArm_p1/J2_Link3.STL; visual mesh filename=package://mycobot_description/urdf/ultraArm_p1/J2_Link3.STL
- added link J3_LIink2, mass 0.0559892080648003; collision mesh filename=package://mycobot_description/urdf/ultraArm_p1/J3_LIink2.STL; visual mesh filename=package://mycobot_description/urdf/ultraArm_p1/J3_LIink2.STL
- link FIX1: geometry collision mesh filename=package://mycobot_description/urdf/ultraArm_p1/FIX1.STL; visual mesh filename=package://mycobot_description/urdf/ultraArm_p1/FIX1.STL
- link FIX2: geometry collision mesh filename=package://mycobot_description/urdf/ultraArm_p1/FIX2.STL; visual mesh filename=package://mycobot_description/urdf/ultraArm_p1/FIX2.STL
- link FIX3: geometry collision mesh filename=package://mycobot_description/urdf/ultraArm_p1/FIX3.STL; visual mesh filename=package://mycobot_description/urdf/ultraArm_p1/FIX3.STL
- link J2_Link1: geometry collision mesh filename=package://mycobot_description/urdf/ultraArm_p1/J2_Link1.STL; visual mesh filename=package://mycobot_description/urdf/ultraArm_p1/J2_Link1.STL
- link J2_Link2: geometry collision mesh filename=package://mycobot_description/urdf/ultraArm_p1/J2_Link2.STL; visual mesh filename=package://mycobot_description/urdf/ultraArm_p1/J2_Link2.STL
- link J2_Link4: geometry collision mesh filename=package://mycobot_description/urdf/ultraArm_p1/J2_Link4.STL; visual mesh filename=package://mycobot_description/urdf/ultraArm_p1/J2_Link4.STL
- link J3_Link1: geometry collision mesh filename=package://mycobot_description/urdf/ultraArm_p1/J3_Link1.STL; visual mesh filename=package://mycobot_description/urdf/ultraArm_p1/J3_Link1.STL
- link J3_Link3: geometry collision mesh filename=package://mycobot_description/urdf/ultraArm_p1/J3_Link3.STL; visual mesh filename=package://mycobot_description/urdf/ultraArm_p1/J3_Link3.STL
- link J3_Link4: geometry collision mesh filename=package://mycobot_description/urdf/ultraArm_p1/J3_Link4.STL; visual mesh filename=package://mycobot_description/urdf/ultraArm_p1/J3_Link4.STL
- link J4_Link: geometry collision mesh filename=package://mycobot_description/urdf/ultraArm_p1/J4_Link.STL; visual mesh filename=package://mycobot_description/urdf/ultraArm_p1/J4_Link.STL
- link base_link: geometry collision mesh filename=package://mycobot_description/urdf/ultraArm_p1/base_link.STL; visual mesh filename=package://mycobot_description/urdf/ultraArm_p1/base_link.STL
Joints:
- removed joint J2-2
- removed joint J2-3
- removed joint J2-4
- removed joint J3-2
- removed joint J3-3
- removed joint J3-4
- added joint J2_2: type revolute, parent J1_LINK, child J2_Link2, origin xyz=-0.0025 -0.024 0.1049 rpy=0 0 0, axis 0 1 0, limit lower=-0.35 upper=1.3962 effort=100 velocity=1, mimic joint=J2 multiplier=1 offset=0
- added joint J2_3: type revolute, parent J2_Link2, child J2_Link3, origin xyz=0 0 0.14 rpy=0 0 0, axis 0 1 0, limit lower=1.3962 upper=0.35 effort=100 velocity=1, mimic joint=J2 multiplier=-1 offset=0
- added joint J2_4: type revolute, parent J2_Link1, child J2_Link4, origin xyz=-0.002409 0.0059 0.13998 rpy=0 0 0, axis 0 1 0, limit lower=-1.3962 upper=0.35 effort=100 velocity=1, mimic joint=J2_3 multiplier=1 offset=0
- added joint J3_2: type revolute, parent FIX3, child J3_LIink2, origin xyz=0 0 0 rpy=0 0 0, axis 0 1 0, limit lower=0 upper=1.92 effort=100 velocity=1, mimic joint=J3 multiplier=1 offset=0
- added joint J3_3: type revolute, parent J3_Link1, child J3_Link3, origin xyz=0.14232 -0.0099 -0.0049908 rpy=0 0 0, axis 0 1 0, limit lower=-1.92 upper=0 effort=100 velocity=1, mimic joint=J3 multiplier=-1 offset=0
- added joint J3_4: type revolute, parent J3_LIink2, child J3_Link4, origin xyz=0.13991 0.005 -0.0050135 rpy=0 0 0, axis 0 1 0, limit lower=-1.92 upper=0 effort=100 velocity=1, mimic joint=J3_3 multiplier=1 offset=0
- joint J1: child J1-LINK -> J1_LINK
- joint J2: parent J1-LINK -> J1_LINK

Commit message: perf(p1-ros):Update URDF joint limits and update function package code.

File: mycobot_description/urdf/ultraArm_p1/ultraArm_p1.urdf (robot description, URDF)
Before this commit: robot firefighter, 15 links, 14 joints
Joints:
- joint J1: limit lower=-2.97 upper=2.97 effort=100 velocity=1 -> lower=-2.87 upper=2.87 effort=100 velocity=1
- joint J2: limit lower=-0.35 upper=1.3962 effort=100 velocity=1 -> lower=-0.31 upper=1.48 effort=100 velocity=1
- joint J2_2: limit lower=-0.35 upper=1.3962 effort=100 velocity=1 -> lower=-0.31 upper=1.48 effort=100 velocity=1
- joint J2_3: limit lower=1.3962 upper=0.35 effort=100 velocity=1 -> lower=1.48 upper=0.31 effort=100 velocity=1
- joint J2_4: limit lower=-1.3962 upper=0.35 effort=100 velocity=1 -> lower=-1.48 upper=0.31 effort=100 velocity=1
- joint J3: limit lower=0 upper=1.92 effort=100 velocity=1 -> lower=0 upper=3.49 effort=100 velocity=1
- joint J3_2: limit lower=0 upper=1.92 effort=100 velocity=1 -> lower=0 upper=3.49 effort=100 velocity=1
- joint J3_3: limit lower=-1.92 upper=0 effort=100 velocity=1 -> lower=-3.49 upper=0 effort=100 velocity=1
- joint J3_4: limit lower=-1.92 upper=0 effort=100 velocity=1 -> lower=-3.49 upper=0 effort=100 velocity=1
- joint J4: limit lower=-3.14 upper=3.14 effort=100 velocity=1 -> lower=-3.12 upper=3.12 effort=100 velocity=1

Commit message: fix(p1-ros1):Fixed some test bugs.

File: mycobot_description/urdf/ultraArm_p1/ultraArm_p1.urdf (robot description, URDF)
Before this commit: robot firefighter, 15 links, 14 joints
Joints:
- joint J3: limit lower=0 upper=3.49 effort=100 velocity=1 -> lower=0 upper=1.91 effort=100 velocity=1
- joint J3_2: limit lower=0 upper=3.49 effort=100 velocity=1 -> lower=0 upper=1.91 effort=100 velocity=1
- joint J3_3: limit lower=-3.49 upper=0 effort=100 velocity=1 -> lower=-1.91 upper=0 effort=100 velocity=1
- joint J3_4: limit lower=-3.49 upper=0 effort=100 velocity=1 -> lower=-1.91 upper=0 effort=100 velocity=1
